File: hardware/Eagle Designs/BBB_OBC/On Board Computer.brd (EAGLE design)
At the start: 90.2 x 95.5 mm, 25 parts, among them J1 MOLEX_503763-0491MOLEX_503763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, J10 503763-0591, J11 503763-0591, J12 503763-0691, J13 MOLEX_503763-0291MOLEX_503763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, J14 MOLEX_503763-0491MOLEX_503763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, J15 MOLEX_503763-0491MOLEX_503763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, J2 MOLEX_503763-0491MOLEX_503763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, J3 503763-0591, J4 503763-0591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

Commit message: Edited payload board, created payload and bbb obc BOM
Connections:
- new net GPIO_FAULT1: H1.1.40
- new net GPIO_FAULT2: H1.1.46
- new net GPIO_SLEEP1: H1.1.42
- new net GPIO_SLEEP2: H1.1.48
- new net GPIO_TRQ1: H1.1.38
- new net GPIO_TRQ2: H1.1.44
Changed lines of the file:
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@@
 <wire x1="76.6362" y1="29.4988" x2="76.635" y2="29.5" width="0.3048" layer="1"/>
+</signal>
+<signal name="GPIO_FAULT1">
+<contactref element="H1" pad="1.40"/>
+</signal>
+<signal name="GPIO_SLEEP1">
+<contactref element="H1" pad="1.42"/>
+</signal>
+<signal name="GPIO_TRQ1">
+<contactref element="H1" pad="1.38"/>
+</signal>
+<signal name="GPIO_FAULT2">
+<contactref element="H1" pad="1.46"/>
+</signal>
+<signal name="GPIO_SLEEP2">
+<contactref element="H1" pad="1.48"/>
+</signal>
+<signal name="GPIO_TRQ2">
+<contactref element="H1" pad="1.44"/>
 </signal>
 </signals>
