File: hardware/Eagle Designs/Antenna/Antenna Board.brd (EAGLE design)
At the start: 100 x 100 mm, 12 parts, among them J1 503763-0591, J10 U.FL-R-SMT-1(01), J2 MOLEX_503763-0491MOLEX_503763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, J3 MOLEX_503763-0491MOLEX_503763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, J4 MOLEX_503763-0291MOLEX_503763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, J5 503763-0591, J6 MOLEX_503763-0491MOLEX_503763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, J7 MOLEX_503763-0491MOLEX_503763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, J8 MOLEX_503763-0291MOLEX_503763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, J9 MOLEX_503763-0291MOLEX_503763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

Commit message: Update Antenna Board.brd
Parts:
- moved U$2 15.0 mm to (35.0, 26.7)
- moved J10 2.22 mm to (50.0, 11.4), turned to 180 degrees
Routing:
- net ANTENNA: track 15.6 -> 26.5 mm
Changed lines of the file:
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@@
 <setting verticaltext="up"/>
 </settings>
-<grid distance="0.2" unitdist="mm" unit="mm" style="lines" multiple="1" display="yes" altdistance="0.1" altunitdist="mm" altunit="mm"/>
+<grid distance="1" unitdist="mm" unit="mm" style="lines" multiple="1" display="yes" altdistance="0.1" altunitdist="mm" altunit="mm"/>
 <layers>
 <layer number="1" name="Top" color="4" fill="1" visible="yes" active="yes"/>
@@
 <wire x1="10" y1="90" x2="0" y2="90" width="0.1524" layer="20"/>
 <wire x1="0" y1="90" x2="0" y2="10" width="0.1524" layer="20"/>
-<hole x="35" y="4.2" drill="3.26"/>
 <hole x="35" y="19.2" drill="3.26"/>
+<hole x="35" y="34.2" drill="3.26"/>
 </plain>
 <attributes>
@@
 <attribute name="TEMPERATURE_RANGE_LOW" value="-40°C" x="20.01" y="25.11" size="1.778" layer="28" rot="MR270" display="off"/>
 </element>
-<element name="J10" library="U.FL-R-SMT-1(01)" package="CONN_-SMT-1(01)" value="U.FL-R-SMT-1(01)" x="52.2" y="11.7" smashed="yes" rot="MR90">
-<attribute name="BUILT_BY" value="EMA_Matt" x="52.2" y="11.7" size="1.778" layer="28" rot="MR90" display="off"/>
-<attribute name="COPYRIGHT" value="Copyright (C) 2018 Accelerated Designs. All rights reserved" x="52.2" y="11.7" size="1.778" layer="28" rot="MR90" display="off"/>
-<attribute name="MANUFACTURER_PART_NUMBER" value="U.FL-R-SMT-1(01)" x="52.2" y="11.7" size="1.778" layer="28" rot="MR90" display="off"/>
-<attribute name="NAME" x="55.0224" y="14.0904" size="1.27" layer="26" ratio="6" rot="SMR270"/>
-<attribute name="SOURCELIBRARY" value="Hirose_12_20_2019" x="52.2" y="11.7" size="1.778" layer="28" rot="MR90" display="off"/>
-<attribute name="VENDOR" value="Hirose" x="52.2" y="11.7" size="1.778" layer="28" rot="MR90" display="off"/>
+<element name="J10" library="U.FL-R-SMT-1(01)" package="CONN_-SMT-1(01)" value="U.FL-R-SMT-1(01)" x="50" y="11.4" smashed="yes" rot="MR180">
+<attribute name="BUILT_BY" value="EMA_Matt" x="50" y="11.4" size="1.778" layer="28" rot="MR180" display="off"/>
+<attribute name="COPYRIGHT" value="Copyright (C) 2018 Accelerated Designs. All rights reserved" x="50" y="11.4" size="1.778" layer="28" rot="MR180" display="off"/>
+<attribute name="MANUFACTURER_PART_NUMBER" value="U.FL-R-SMT-1(01)" x="50" y="11.4" size="1.778" layer="28" rot="MR180" display="off"/>
+<attribute name="NAME" x="52.3904" y="8.5776" size="1.27" layer="26" ratio="6" rot="SMR0"/>
+<attribute name="SOURCELIBRARY" value="Hirose_12_20_2019" x="50" y="11.4" size="1.778" layer="28" rot="MR180" display="off"/>
+<attribute name="VENDOR" value="Hirose" x="50" y="11.4" size="1.778" layer="28" rot="MR180" display="off"/>
 </element>
 <element name="J8" library="Molex - 503763-0291" package="MOLEX_503763-0291_0" value="MOLEX_503763-0291MOLEX_503763-0291_0_0" x="16.2" y="39.6" smashed="yes" rot="MR270">
@@
 <attribute name="VENDOR" value="Molex Connector Corporation" x="84.2" y="76.2" size="1.778" layer="28" rot="MR270" display="off"/>
 </element>
-<element name="U$2" library="Antenna_Pad" package="ANTENNA_PAD" value="ANTENNA_PAD" x="35" y="11.7" smashed="yes"/>
+<element name="U$2" library="Antenna_Pad" package="ANTENNA_PAD" value="ANTENNA_PAD" x="35" y="26.7" smashed="yes"/>
 <element name="U$3" library="Burn_Wire" package="BURNWIRE" value="BURNWIRE" x="35" y="93" smashed="yes"/>
 </elements>
@@
 <contactref element="J10" pad="3"/>
 <contactref element="U$2" pad="1"/>
-<wire x1="35" y1="11.7" x2="46.2" y2="11.7" width="0.508" layer="1"/>
-<wire x1="50.6039" y1="11.7" x2="46.2" y2="11.7" width="0.508" layer="16"/>
-<via x="46.2" y="11.7" extent="1-16" drill="0.35"/>
+<wire x1="35" y1="26.7" x2="46.3" y2="26.7" width="0.508" layer="1"/>
+<wire x1="46.3" y1="26.7" x2="50" y2="23" width="0.508" layer="1"/>
+<wire x1="50" y1="12.9961" x2="50" y2="23" width="0.508" layer="16"/>
+<via x="50" y="23" extent="1-16" drill="0.35"/>
 </signal>
 <signal name="VCC_BURN">
