File: hardware/Eagle Designs/Antenna/Antenna Board v2.brd (EAGLE design)
At the start: 100 x 100 mm, 14 parts, among them J1 503763-0591, J10 U.FL-R-SMT-1(01), J11 U.FL-R-SMT-1(01), J12 U.FL-R-SMT-1(01), J2 MOLEX_503763-0491MOLEX_503763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, J3 MOLEX_503763-0491MOLEX_503763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, J4 MOLEX_503763-0291MOLEX_503763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, J5 503763-0591, J6 MOLEX_503763-0491MOLEX_503763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, J7 MOLEX_503763-0491MOLEX_503763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

Commit message: Updated antenna and solar panel boards
Parts:
- J1, J5: device Molex - 503763-0591:CONN_5037630591_MOL -> Improved Molex 503763-0591:CONN_5037630591_MOL
Connections:
- net GND: now also J1.6, J1.7, J5.6, J5.7
Changed lines of the file:
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@@
 </autorouter>
 <elements>
-<element name="J1" library="Molex - 503763-0591" package="CONN_5037630591_MOL" value="503763-0591" x="77.6" y="69.2" smashed="yes" rot="R270">
+<element name="J1" library="Improved Molex 503763-0591" package="CONN_5037630591_MOL" value="503763-0591" x="77.6" y="69.2" smashed="yes" rot="R270">
 <attribute name="BUILT_BY" value="EMA_Cory" x="48.39" y="46.34" size="1.778" layer="27" rot="R270" display="off"/>
 <attribute name="COPYRIGHT" value="Copyright (C) 2018 Accelerated Designs. All rights reserved" x="48.39" y="46.34" size="1.778" layer="27" rot="R270" display="off"/>
@@
 <attribute name="VOLTAGE_RATING" value="150V" x="66.1" y="44.3" size="1.778" layer="28" rot="MR270" display="off"/>
 </element>
-<element name="J5" library="Molex - 503763-0591" package="CONN_5037630591_MOL" value="503763-0591" x="65.6" y="69.1" smashed="yes" rot="MR90">
+<element name="J5" library="Improved Molex 503763-0591" package="CONN_5037630591_MOL" value="503763-0591" x="65.6" y="69.1" smashed="yes" rot="MR90">
 <attribute name="BUILT_BY" value="EMA_Cory" x="65.6" y="61.1" size="1.778" layer="28" rot="MR90" display="off"/>
 <attribute name="COPYRIGHT" value="Copyright (C) 2018 Accelerated Designs. All rights reserved" x="65.6" y="61.1" size="1.778" layer="28" rot="MR90" display="off"/>
@@
 <signals>
 <signal name="VCC_MICRO">
-<contactref element="J1" pad="1"/>
 <contactref element="J5" pad="5"/>
 <via x="66.6" y="71.1" extent="1-16" drill="0.35"/>
@@
 <wire x1="79.7608" y1="71.1" x2="79.8608" y2="71.2" width="0.508" layer="1"/>
 <wire x1="67.8608" y1="71.1" x2="66.6" y2="71.1" width="0.508" layer="16"/>
+<contactref element="J1" pad="1"/>
 </signal>
 <signal name="D+_MICRO">
-<contactref element="J1" pad="2"/>
 <contactref element="J5" pad="4"/>
 <via x="66.6" y="70.1" extent="1-16" drill="0.35"/>
@@
 <wire x1="79.7608" y1="70.1" x2="79.8608" y2="70.2" width="0.508" layer="1"/>
 <wire x1="67.8608" y1="70.1" x2="66.6" y2="70.1" width="0.508" layer="16"/>
+<contactref element="J1" pad="2"/>
 </signal>
 <signal name="D-_MICRO">
-<contactref element="J1" pad="3"/>
 <contactref element="J5" pad="3"/>
 <via x="66.6" y="69.1" extent="1-16" drill="0.35"/>
@@
 <wire x1="79.7608" y1="69.1" x2="66.6" y2="69.1" width="0.508" layer="1"/>
 <wire x1="67.8608" y1="69.1" x2="66.6" y2="69.1" width="0.508" layer="16"/>
+<contactref element="J1" pad="3"/>
 </signal>
 <signal name="ID_MICRO">
-<contactref element="J1" pad="4"/>
 <contactref element="J5" pad="2"/>
 <via x="66.6" y="68.1" extent="1-16" drill="0.35"/>
@@
 <wire x1="79.7608" y1="68.1" x2="79.8608" y2="68.2" width="0.508" layer="1"/>
 <wire x1="67.8608" y1="68.1" x2="66.74185" y2="68.1" width="0.508" layer="16"/>
-<wire x1="79.7608" y1="68.1" x2="66.74185" y2="68.1" width="0" layer="19" extent="16-16"/>
+<contactref element="J1" pad="4"/>
+<wire x1="66.74185" y1="68.1" x2="66.6" y2="68.1" width="0" layer="19" extent="16-16"/>
 </signal>
 <signal name="VCC_HOST">
@@
 <wire x1="28.255" y1="42.875" x2="46.0544" y2="42.875" width="0.508" layer="16"/>
 <wire x1="46.0544" y1="42.875" x2="46.5295" y2="42.3999" width="0.508" layer="16"/>
+<contactref element="J1" pad="7"/>
+<contactref element="J1" pad="6"/>
+<contactref element="J5" pad="7"/>
+<contactref element="J5" pad="6"/>
 </signal>
 <signal name="ANTENNA">
