File: hardware/Eagle Designs/Antenna/Antenna Board v5.0.sch (EAGLE design)
At the start: 17 parts, among them J1 5037630291, J10 MCX-J-P-X-ST-TH1, J11 U.FL-R-SMT-1(01), J12 MCX-J-P-X-ST-TH1, J13 MCX-J-P-X-ST-TH1, J14 MOLEX_503763-0491MOLEX_503763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, J16 ARJM11C7-104-AB-EW2, J17 UJ2-MIBH-G-SMT-TR, J18 M55-6001642R, J2 503763-0591, J3 MOLEX_503763-0491MOLEX_503763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, J4 MOLEX_503763-0291MOLEX_503763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, J9 MOLEX_503763-0291MOLEX_503763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

Commit message: Updated Artemis v2 EAGLE library, solar panel board, and antenna board
Parts:
- removed J14: MOLEX_503763-0491MOLEX_503763-0491_0_0, Molex - 503763-0491:MOLEX_503763-0491MOLEX_503763-0491_0_0
- removed J16: ARJM11C7-104-AB-EW2, ARJM11C7-104-AB-EW2:ARJM11C7-104-AB-EW2
- removed J17: UJ2-MIBH-G-SMT-TR, UJ2-MIBH-G-SMT-TR:UJ2-MIBH-G-SMT-TR
- removed J18: M55-6001642R, M55-60X1642R:M55-6001642R
- added J5: ARJM11C7-104-AB-EW2, ARJM11C7-104-AB-EW2:ARJM11C7-104-AB-EW2
- added J6: MOLEX_503763-0291MOLEX_503763-0291_0_0, Molex - 503763-0291:MOLEX_503763-0291MOLEX_503763-0291_0_0
- added J7: MOLEX_503763-0491MOLEX_503763-0491_0_0, Molex - 503763-0491:MOLEX_503763-0491MOLEX_503763-0491_0_0
- added J8: UJ2-MIBH-G-SMT-TR, UJ2-MIBH-G-SMT-TR:UJ2-MIBH-G-SMT-TR
- J1: value 5037630291 -> M55-6001642R; device Molex_503763-0291:5037630291 -> M55-6001642R:M55-6001642R
- J10: value MCX-J-P-X-ST-TH1 -> U.FL-R-SMT-1(01); device MCX-J-P-X-ST-TH1:MCX-J-P-X-ST-TH1 -> U.FL-R-SMT-1(01):U.FL-R-SMT-1(01)
- J11: value U.FL-R-SMT-1(01) -> MCX-J-P-X-ST-TH1; device U.FL-R-SMT-1(01):U.FL-R-SMT-1(01) -> MCX-J-P-X-ST-TH1:MCX-J-P-X-ST-TH1
- J2: value 503763-0591 -> 5037630291; device Molex - 503763-0591:503763-0591 -> Molex_503763-0291:5037630291
- J3: value MOLEX_503763-0491MOLEX_503763-0491_0_0 -> 503763-0591; device Molex - 503763-0491:MOLEX_503763-0491MOLEX_503763-0491_0_0 -> Molex - 503763-0591:503763-0591
- J4: value MOLEX_503763-0291MOLEX_503763-0291_0_0 -> MOLEX_503763-0491MOLEX_503763-0491_0_0; device Molex - 503763-0291:MOLEX_503763-0291MOLEX_503763-0291_0_0 -> Molex - 503763-0491:MOLEX_503763-0491MOLEX_503763-0491_0_0
Connections:
- net 5V: now also J1.9, J7.4, J8.VCC; no longer J14.4, J17.VCC, J18.9
- net ANTENNA1: now also J12.1; no longer J10.1
- net D+: now also J1.13, J7.2, J8.D+; no longer J14.2, J17.D+, J18.13
- net D-: now also J1.11, J7.3, J8.D-; no longer J14.3, J17.D-, J18.11
- net GND: now also J1.1, J1.GND, J10.1, J2.3, J3.4, J3.6, J3.7, J6.2, J6.MNT_1, J6.MNT_2, J7.1, J7.MNT_1, J7.MNT_2, J8.GND, J8.SHIELD; no longer J1.4, J11.1, J14.1, J14.MNT_1, J14.MNT_2, J17.GND, J17.SHIELD, J18.1, J18.17, J18.3, J2.6, J2.7, J3.MNT_1, J3.MNT_2, J4.2
- net ID: now also J8.ID; no longer J17.ID
- net ORION-SPACE: now also J10.3, J11.1; no longer J11.3, J12.1
- net RBF1: now also J1.7, J2.1; no longer J1.1, J18.7
- net RBF2: now also J1.5, J2.2; no longer J1.2, J18.5
- net RESET: now also J1.2, J3.1; no longer J18.2, J2.1
- net RX+: now also J1.14, J4.3, J5.3; no longer J16.3, J18.14, J3.3
- net RX-: now also J1.16, J4.4, J5.6; no longer J16.6, J18.16, J3.4
- net TCK: now also J1.4, J3.2; no longer J18.4, J2.2
- net TMS: now also J1.6, J3.3; no longer J18.6, J2.3
- net TX+: now also J1.10, J4.1, J5.1; no longer J16.1, J18.10, J3.1
- net TX-: now also J1.12, J4.2, J5.2; no longer J16.2, J18.12, J3.2
- net VCC_BATT: now also J1.15, J6.1; no longer J18.15, J4.1
- net VRTREF: now also J1.8, J3.5; no longer J18.8, J2.5
Other:
- note added: "Antenna header"
- moved on the sheet: J12, J13, J9
