File: hardware/Eagle Designs/Payload/Payload.sch (EAGLE design)
At the start: 81 parts, among them J1 503763-0591, J2 503763-0591, J3 MOLEX_503763-0491MOLEX_503763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, J4 503763-0691, J5 MOLEX_503763-0291MOLEX_503763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, J6 503763-0691, J7 503763-0691, M1 BSZ100N06LS3, M2 BSZ100N06LS3, M3 BSZ033NE2LS5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

Commit message: Edited payload board, created payload and bbb obc BOM
Parts:
- added X1: C25582-40G-M36-0A, Adafruit - C25582-40G-M36-0A:C25582-40G-M36-0A
Connections:
- removed net 3V3: R13.2, R16.2
- removed net 5V: C14.2, C18.2, C19.2, C20.2, U1.VM, U2.VM
- net +3V3_BUS: now also R13.2, R16.2
- net +3V3_VCC: now also X1.P$1; no longer X2-1.1
- net +5V_BUS: now also C14.2, C18.2, C19.2, C20.2, U1.VM, U2.VM
- net GPIO12: now also X1.P$32; no longer X2-32.1
- net GPIO13: now also X1.P$33; no longer X2-33.1
- net GPIO16: now also X1.P$36; no longer X2-36.1
- net GPIO17: now also X1.P$11; no longer X2-11.1
- net GPIO19: now also X1.P$35; no longer X2-35.1
- net GPIO20: now also X1.P$38; no longer X2-38.1
- net GPIO21: now also X1.P$40; no longer X2-40.1
- net GPIO22: now also X1.P$15; no longer X2-15.1
- net GPIO23: now also X1.P$16; no longer X2-16.1
- net GPIO24: now also X1.P$18; no longer X2-18.1
- net GPIO25: now also X1.P$22; no longer X2-22.1
- net GPIO26: now also X1.P$37; no longer X2-37.1
- net GPIO27: now also X1.P$13; no longer X2-13.1
- net GPIO6: now also X1.P$31; no longer X2-31.1
- net GPIO_FAULT1: now also H1.1.40; no longer H1.1.47
- net GPIO_FAULT2: now also H1.1.46; no longer H1.1.51
- net GPIO_SLEEP1: now also H1.1.42; no longer H1.1.49
- net GPIO_SLEEP2: now also H1.1.48; no longer H1.1.52
- net GPIO_TRQ1: now also H1.1.38; no longer H1.1.48
- net GPIO_TRQ2: now also H1.1.44; no longer H1.1.50
- net SCL1_I2C: now also X1.P$5; no longer X2-5.1
- net SDA1_I2C: now also X1.P$3; no longer X2-3.1
- net SPI0_CE0_N: now also X1.P$24; no longer X2-24.1
- net SPI0_CE1_N: now also X1.P$26; no longer X2-26.1
- net SPI0_MISO: now also X1.P$21; no longer X2-21.1
- net SPI0_MOSI: now also X1.P$19; no longer X2-19.1
- net SPI0_SCLK: now also X1.P$23; no longer X2-23.1
Other:
- moved on the sheet: X2-1, X2-10, X2-11, X2-12, X2-13, X2-14, X2-15, X2-16, X2-17, X2-18, X2-19, X2-2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

Commit message: Update payload board
Parts:
- added J8, J9: MOLEX_503763-0491MOLEX_503763-0491_0_0, Molex - 503763-0491:MOLEX_503763-0491MOLEX_503763-0491_0_0
Connections:
- net 12V_SW1: now also J4.3; no longer J4.1
- net 3V3_SW1: now also J3.1; no longer J3.2
- net 5V_SW3: now also J4.1; no longer J4.3
- net 5V_SW4: now also J3.2; no longer J3.1
- net IN1: now also H1.1.26
- net IN2: now also H1.1.25
- net IN3: now also H1.1.23
- net IN4: now also H1.1.24
- net IN5: now also H1.1.30
- net IN6: now also H1.1.29
- net IN7: now also H1.1.27
- net IN8: now also H1.1.28
Changed lines of the file:
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@@
 <part name="X1" library="Adafruit - C25582-40G-M36-0A" deviceset="C25582-40G-M36-0A" device=""/>
 <part name="X2" library="con-samtec" library_urn="urn:adsk.eagle:library:184" deviceset="SSW-120-02-G" device="-D"/>
+<part name="J8" library="Molex - 503763-0491" deviceset="MOLEX_503763-0491" device="MOLEX_503763-0491_0_0"/>
+<part name="J9" library="Molex - 503763-0491" deviceset="MOLEX_503763-0491" device="MOLEX_503763-0491_0_0"/>
 </parts>
 <sheets>
@@
 <instance part="X2" gate="-40" x="365.76" y="185.42" smashed="yes">
 <attribute name="NAME" x="362.712" y="186.182" size="1.524" layer="95" rot="R180"/>
+</instance>
+<instance part="J8" gate="G$0" x="281.94" y="71.12" smashed="yes">
+<attribute name="NAME" x="284.48" y="68.58" size="2.54" layer="95" align="top-left"/>
+</instance>
+<instance part="J9" gate="G$0" x="307.34" y="71.12" smashed="yes">
+<attribute name="NAME" x="309.88" y="68.58" size="2.54" layer="95" align="top-left"/>
 </instance>
 </instances>
@@
 </segment>
 <segment>
-<pinref part="J4" gate="A" pin="1"/>
-<wire x1="347.98" y1="134.62" x2="345.44" y2="134.62" width="0.1524" layer="91"/>
-<label x="345.44" y="134.62" size="1.778" layer="95" rot="MR0"/>
+<wire x1="347.98" y1="129.54" x2="345.44" y2="129.54" width="0.1524" layer="91"/>
+<label x="345.44" y="129.54" size="1.778" layer="95" rot="MR0"/>
+<pinref part="J4" gate="A" pin="3"/>
 </segment>
 </net>
@@
 </segment>
 <segment>
-<pinref part="J4" gate="A" pin="3"/>
-<wire x1="347.98" y1="129.54" x2="345.44" y2="129.54" width="0.1524" layer="91"/>
-<label x="345.44" y="129.54" size="1.778" layer="95" rot="MR0"/>
+<wire x1="347.98" y1="134.62" x2="345.44" y2="134.62" width="0.1524" layer="91"/>
+<label x="345.44" y="134.62" size="1.778" layer="95" rot="MR0"/>
+<pinref part="J4" gate="A" pin="1"/>
 </segment>
 </net>
@@
 </segment>
 <segment>
-<pinref part="J3" gate="G$0" pin="1"/>
-<wire x1="314.96" y1="139.7" x2="317.5" y2="139.7" width="0.1524" layer="91"/>
-<label x="317.5" y="139.7" size="1.778" layer="95"/>
+<wire x1="314.96" y1="134.62" x2="317.5" y2="134.62" width="0.1524" layer="91"/>
+<label x="317.5" y="134.62" size="1.778" layer="95"/>
+<pinref part="J3" gate="G$0" pin="2"/>
 </segment>
 </net>
@@
 </segment>
 <segment>
-<pinref part="J3" gate="G$0" pin="2"/>
-<wire x1="314.96" y1="134.62" x2="317.5" y2="134.62" width="0.1524" layer="91"/>
-<label x="317.5" y="134.62" size="1.778" layer="95"/>
+<wire x1="314.96" y1="139.7" x2="317.5" y2="139.7" width="0.1524" layer="91"/>
+<label x="317.5" y="139.7" size="1.778" layer="95"/>
+<pinref part="J3" gate="G$0" pin="1"/>
 </segment>
 </net>
@@
 <pinref part="U1" gate="G$1" pin="IN4"/>
 </segment>
+<segment>
+<pinref part="H1" gate="G$1" pin="1.24"/>
+<wire x1="99.06" y1="187.96" x2="106.68" y2="187.96" width="0.1524" layer="91"/>
+<label x="106.68" y="187.96" size="1.778" layer="95"/>
+</segment>
 </net>
 <net name="TORQUE_1A" class="0">
@@
 <label x="218.44" y="129.54" size="1.778" layer="95" rot="MR0"/>
 </segment>
+<segment>
+<pinref part="H1" gate="G$1" pin="1.26"/>
+<wire x1="99.06" y1="185.42" x2="106.68" y2="185.42" width="0.1524" layer="91"/>
+<label x="106.68" y="185.42" size="1.778" layer="95"/>
+</segment>
 </net>
 <net name="IN2" class="0">
@@
 <pinref part="U1" gate="G$1" pin="IN2"/>
 </segment>
+<segment>
+<pinref part="H1" gate="G$1" pin="1.25"/>
+<wire x1="71.12" y1="185.42" x2="63.5" y2="185.42" width="0.1524" layer="91"/>
+<label x="63.5" y="185.42" size="1.778" layer="95" rot="MR0"/>
+</segment>
 </net>
 <net name="IN3" class="0">
@@
 <label x="218.44" y="124.46" size="1.778" layer="95" rot="MR0"/>
 <pinref part="U1" gate="G$1" pin="IN3"/>
+</segment>
+<segment>
+<pinref part="H1" gate="G$1" pin="1.23"/>
+<wire x1="71.12" y1="187.96" x2="63.5" y2="187.96" width="0.1524" layer="91"/>
+<label x="63.5" y="187.96" size="1.778" layer="95" rot="MR0"/>
 </segment>
 </net>
@@
 <pinref part="U2" gate="G$1" pin="IN4"/>
 </segment>
+<segment>
+<pinref part="H1" gate="G$1" pin="1.28"/>
+<wire x1="99.06" y1="182.88" x2="106.68" y2="182.88" width="0.1524" layer="91"/>
+<label x="106.68" y="182.88" size="1.778" layer="95"/>
+</segment>
 </net>
 <net name="TORQUE_3A" class="0">
@@
 <label x="218.44" y="63.5" size="1.778" layer="95" rot="MR0"/>
 </segment>
+<segment>
+<pinref part="H1" gate="G$1" pin="1.30"/>
+<wire x1="99.06" y1="180.34" x2="106.68" y2="180.34" width="0.1524" layer="91"/>
+<label x="106.68" y="180.34" size="1.778" layer="95"/>
+</segment>
 </net>
 <net name="IN6" class="0">
@@
 <pinref part="U2" gate="G$1" pin="IN2"/>
 </segment>
+<segment>
+<pinref part="H1" gate="G$1" pin="1.29"/>
+<wire x1="71.12" y1="180.34" x2="63.5" y2="180.34" width="0.1524" layer="91"/>
+<label x="63.5" y="180.34" size="1.778" layer="95" rot="MR0"/>
+</segment>
 </net>
 <net name="IN7" class="0">
@@
 <pinref part="U2" gate="G$1" pin="IN3"/>
 </segment>
-</net>
+<segment>
+<pinref part="H1" gate="G$1" pin="1.27"/>
+<wire x1="71.12" y1="182.88" x2="63.5" y2="182.88" width="0.1524" layer="91"/>
+<label x="63.5" y="182.88" size="1.778" layer="95" rot="MR0"/>
+</segment>
+</net>

Commit message: Payload board changes
Connections:
- net GND: now also J7.6; no longer J6.6
- net GPIO17: now also J6.1; no longer J7.1
- net GPIO22: now also J6.4; no longer J7.4
- net GPIO23: now also J6.3; no longer J7.3
- net GPIO24: now also J6.5; no longer J7.5
- net GPIO25: now also J6.6; no longer J7.6
- net GPIO27: now also J6.2; no longer J7.2
- net SPI0_CE0_N: now also J7.3; no longer J6.3
- net SPI0_CE1_N: now also J7.5; no longer J6.5
- net SPI0_MISO: now also J7.2; no longer J6.2
- net SPI0_MOSI: now also J7.1; no longer J6.1
- net SPI0_SCLK: now also J7.4; no longer J6.4
- net TORQUE_1A: now also J8.1
- net TORQUE_1B: now also J8.2
- net TORQUE_2A: now also J8.4
- net TORQUE_2B: now also J8.3
- net TORQUE_3A: now also J9.1
- net TORQUE_3B: now also J9.2
- net TORQUE_4A: now also J9.4
- net TORQUE_4B: now also J9.3
Other:
- moved on the sheet: J5, J6, J7, J8, J9

Commit message: Payload board changes
Connections:
- net IN1: now also H1.1.24; no longer H1.1.26
- net IN2: now also H1.1.23; no longer H1.1.25
- net IN3: now also H1.1.25; no longer H1.1.23
- net IN4: now also H1.1.26; no longer H1.1.24
- net IN5: now also H1.1.28; no longer H1.1.30
- net IN6: now also H1.1.27; no longer H1.1.29
- net IN7: now also H1.1.29; no longer H1.1.27
- net IN8: now also H1.1.30; no longer H1.1.28
Changed lines of the file:
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@@
 </segment>
 <segment>
-<pinref part="H1" gate="G$1" pin="1.24"/>
-<wire x1="99.06" y1="187.96" x2="106.68" y2="187.96" width="0.1524" layer="91"/>
-<label x="106.68" y="187.96" size="1.778" layer="95"/>
+<wire x1="99.06" y1="185.42" x2="106.68" y2="185.42" width="0.1524" layer="91"/>
+<label x="106.68" y="185.42" size="1.778" layer="95"/>
+<pinref part="H1" gate="G$1" pin="1.26"/>
 </segment>
 </net>
@@
 </segment>
 <segment>
-<pinref part="H1" gate="G$1" pin="1.26"/>
-<wire x1="99.06" y1="185.42" x2="106.68" y2="185.42" width="0.1524" layer="91"/>
-<label x="106.68" y="185.42" size="1.778" layer="95"/>
+<wire x1="99.06" y1="187.96" x2="106.68" y2="187.96" width="0.1524" layer="91"/>
+<label x="106.68" y="187.96" size="1.778" layer="95"/>
+<pinref part="H1" gate="G$1" pin="1.24"/>
 </segment>
 </net>
@@
 </segment>
 <segment>
-<pinref part="H1" gate="G$1" pin="1.25"/>
-<wire x1="71.12" y1="185.42" x2="63.5" y2="185.42" width="0.1524" layer="91"/>
-<label x="63.5" y="185.42" size="1.778" layer="95" rot="MR0"/>
+<wire x1="71.12" y1="187.96" x2="63.5" y2="187.96" width="0.1524" layer="91"/>
+<label x="63.5" y="187.96" size="1.778" layer="95" rot="MR0"/>
+<pinref part="H1" gate="G$1" pin="1.23"/>
 </segment>
 </net>
@@
 </segment>
 <segment>
-<pinref part="H1" gate="G$1" pin="1.23"/>
-<wire x1="71.12" y1="187.96" x2="63.5" y2="187.96" width="0.1524" layer="91"/>
-<label x="63.5" y="187.96" size="1.778" layer="95" rot="MR0"/>
+<wire x1="71.12" y1="185.42" x2="63.5" y2="185.42" width="0.1524" layer="91"/>
+<label x="63.5" y="185.42" size="1.778" layer="95" rot="MR0"/>
+<pinref part="H1" gate="G$1" pin="1.25"/>
 </segment>
 </net>
@@
 </segment>
 <segment>
-<pinref part="H1" gate="G$1" pin="1.28"/>
-<wire x1="99.06" y1="182.88" x2="106.68" y2="182.88" width="0.1524" layer="91"/>
-<label x="106.68" y="182.88" size="1.778" layer="95"/>
+<wire x1="99.06" y1="180.34" x2="106.68" y2="180.34" width="0.1524" layer="91"/>
+<label x="106.68" y="180.34" size="1.778" layer="95"/>
+<pinref part="H1" gate="G$1" pin="1.30"/>
 </segment>
 </net>
@@
 </segment>
 <segment>
-<pinref part="H1" gate="G$1" pin="1.30"/>
-<wire x1="99.06" y1="180.34" x2="106.68" y2="180.34" width="0.1524" layer="91"/>
-<label x="106.68" y="180.34" size="1.778" layer="95"/>
+<wire x1="99.06" y1="182.88" x2="106.68" y2="182.88" width="0.1524" layer="91"/>
+<label x="106.68" y="182.88" size="1.778" layer="95"/>
+<pinref part="H1" gate="G$1" pin="1.28"/>
 </segment>
 </net>
@@
 </segment>
 <segment>
-<pinref part="H1" gate="G$1" pin="1.29"/>
-<wire x1="71.12" y1="180.34" x2="63.5" y2="180.34" width="0.1524" layer="91"/>
-<label x="63.5" y="180.34" size="1.778" layer="95" rot="MR0"/>
+<wire x1="71.12" y1="182.88" x2="63.5" y2="182.88" width="0.1524" layer="91"/>
+<label x="63.5" y="182.88" size="1.778" layer="95" rot="MR0"/>
+<pinref part="H1" gate="G$1" pin="1.27"/>
 </segment>
 </net>
@@
 </segment>
 <segment>
-<pinref part="H1" gate="G$1" pin="1.27"/>
-<wire x1="71.12" y1="182.88" x2="63.5" y2="182.88" width="0.1524" layer="91"/>
-<label x="63.5" y="182.88" size="1.778" layer="95" rot="MR0"/>
-</segment>
-</net>
+<wire x1="71.12" y1="180.34" x2="63.5" y2="180.34" width="0.1524" layer="91"/>
+<label x="63.5" y="180.34" size="1.778" layer="95" rot="MR0"/>
+<pinref part="H1" gate="G$1" pin="1.29"/>
+</segment>
+</net>

Commit message: Added values to resistors and capacitors
Payload - added 3.3k value to pullup resistors for H-bridges
Solar Panel Board - added 0.1uF value to capacitor for temp sensor
Parts:
- R13, R16: value (none) -> 3.3k
Changed lines of the file:
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@@
 <part name="C18" library="HSFL_Main_Library" deviceset="CAP" device="0805" value="0.1 μF"/>
 <part name="GND1" library="SparkFun-PowerSymbols" library_urn="urn:adsk.eagle:library:530" deviceset="GND" device=""/>
-<part name="R13" library="HSFL_Main_Library" deviceset="RESISTOR" device="0805-RES"/>
+<part name="R13" library="HSFL_Main_Library" deviceset="RESISTOR" device="0805-RES" value="3.3k"/>
 <part name="GND18" library="SparkFun-PowerSymbols" library_urn="urn:adsk.eagle:library:530" deviceset="GND" device=""/>
 <part name="U2" library="DRV8847PWPR" deviceset="DRV8847PWPR" device=""/>
@@
 <part name="C20" library="HSFL_Main_Library" deviceset="CAP" device="0805" value="0.1 μF"/>
 <part name="GND19" library="SparkFun-PowerSymbols" library_urn="urn:adsk.eagle:library:530" deviceset="GND" device=""/>
-<part name="R16" library="HSFL_Main_Library" deviceset="RESISTOR" device="0805-RES"/>
+<part name="R16" library="HSFL_Main_Library" deviceset="RESISTOR" device="0805-RES" value="3.3k"/>
 <part name="GND24" library="SparkFun-PowerSymbols" library_urn="urn:adsk.eagle:library:530" deviceset="GND" device=""/>
 <part name="J1" library="Molex - 503763-0591" deviceset="503763-0591" device=""/>

Commit message: Updated BOMs and edited Solar Panel Board v2
Parts:
- C14, C19: value 10 μF -> 10uF
- C18, C20: value 0.1 μF -> 0.1uF
- R11, R12, R14, R15: value 330 mΩ -> 330m
Changed lines of the file:
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@@
 <part name="C13" library="HSFL_Main_Library" deviceset="CAP" device="0805" value="4.7uF"/>
 <part name="U1" library="DRV8847PWPR" deviceset="DRV8847PWPR" device=""/>
-<part name="R11" library="HSFL_Main_Library" deviceset="RESISTOR" device="0805-RES" value="330 mΩ"/>
-<part name="R12" library="HSFL_Main_Library" deviceset="RESISTOR" device="0805-RES" value="330 mΩ"/>
-<part name="C14" library="HSFL_Main_Library" deviceset="CAP" device="0805" value="10 μF"/>
-<part name="C18" library="HSFL_Main_Library" deviceset="CAP" device="0805" value="0.1 μF"/>
+<part name="R11" library="HSFL_Main_Library" deviceset="RESISTOR" device="0805-RES" value="330m"/>
+<part name="R12" library="HSFL_Main_Library" deviceset="RESISTOR" device="0805-RES" value="330m"/>
+<part name="C14" library="HSFL_Main_Library" deviceset="CAP" device="0805" value="10uF"/>
+<part name="C18" library="HSFL_Main_Library" deviceset="CAP" device="0805" value="0.1uF"/>
 <part name="GND1" library="SparkFun-PowerSymbols" library_urn="urn:adsk.eagle:library:530" deviceset="GND" device=""/>
 <part name="R13" library="HSFL_Main_Library" deviceset="RESISTOR" device="0805-RES" value="3.3k"/>
 <part name="GND18" library="SparkFun-PowerSymbols" library_urn="urn:adsk.eagle:library:530" deviceset="GND" device=""/>
 <part name="U2" library="DRV8847PWPR" deviceset="DRV8847PWPR" device=""/>
-<part name="R14" library="HSFL_Main_Library" deviceset="RESISTOR" device="0805-RES" value="330 mΩ"/>
-<part name="R15" library="HSFL_Main_Library" deviceset="RESISTOR" device="0805-RES" value="330 mΩ"/>
-<part name="C19" library="HSFL_Main_Library" deviceset="CAP" device="0805" value="10 μF"/>
-<part name="C20" library="HSFL_Main_Library" deviceset="CAP" device="0805" value="0.1 μF"/>
+<part name="R14" library="HSFL_Main_Library" deviceset="RESISTOR" device="0805-RES" value="330m"/>
+<part name="R15" library="HSFL_Main_Library" deviceset="RESISTOR" device="0805-RES" value="330m"/>
+<part name="C19" library="HSFL_Main_Library" deviceset="CAP" device="0805" value="10uF"/>
+<part name="C20" library="HSFL_Main_Library" deviceset="CAP" device="0805" value="0.1uF"/>
 <part name="GND19" library="SparkFun-PowerSymbols" library_urn="urn:adsk.eagle:library:530" deviceset="GND" device=""/>
 <part name="R16" library="HSFL_Main_Library" deviceset="RESISTOR" device="0805-RES" value="3.3k"/>
