File: hardware/Eagle Designs/Solar Panel Board/Solar Panel Board v2.brd (EAGLE design)
At the start: 82.4 x 96.7 mm, 44 parts, among them J1 MOLEX_503763-0291MOLEX_503763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, J2 MOLEX_503763-0491MOLEX_503763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, J3 MOLEX_503763-0291MOLEX_503763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, U1 TMP36GSZ, U2 INA219BIDR

Commit message: Updated BOMs and edited Solar Panel Board v2
Parts:
- C1: value (none) -> 0.1uF
Changed lines of the file:
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@@
 <attribute name="TEMPERATURE_RANGE_LOW" value="-40°C" x="24.6" y="75.4" size="1.778" layer="28" rot="MR0" display="off"/>
 </element>
-<element name="C1" library="HSFL_Main_Library" package="0805" value="" x="3.5" y="10.6" smashed="yes" rot="MR0">
+<element name="C1" library="HSFL_Main_Library" package="0805" value="0.1uF" x="3.5" y="10.6" smashed="yes" rot="MR0">
 <attribute name="NAME" x="2.678" y="11.6795" size="0.8128" layer="26" font="vector" ratio="15" rot="SMR0"/>
 <attribute name="VALUE" x="5.278" y="8.5045" size="0.8128" layer="28" font="vector" ratio="15" rot="SMR0"/>

Commit message: Add files via upload
Edited Solar Panel Board v2
Connections:
- removed net VIN-: R3.2, U2.7
- net GND: now also R3.2, U2.7
Routing:
- net VIN-: track 6.37 -> 0.00 mm
- net GND: track 0.00 -> 6.37 mm
Changed lines of the file:
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@@
 <contactref element="U2" pad="6"/>
 <contactref element="C2" pad="2"/>
+<contactref element="U2" pad="7"/>
+<contactref element="R3" pad="2"/>
+<wire x1="64.93" y1="33.035" x2="60.465" y2="33.035" width="0.508" layer="16"/>
+<wire x1="60.465" y1="33.035" x2="59.4" y2="34.1" width="0.508" layer="16"/>
+<wire x1="59.4" y1="34.1" x2="59.4" y2="34.5" width="0.1524" layer="16"/>
 </signal>
 <signal name="VCC">
@@
 <contactref element="U2" pad="2"/>
 <contactref element="U$1" pad="1"/>
-<wire x1="75.5" y1="33" x2="72.8" y2="33" width="0.1524" layer="16"/>
-<wire x1="72.8" y1="33" x2="69.905" y2="33" width="0.1524" layer="16"/>
+<wire x1="75.5" y1="33" x2="72.8" y2="33" width="0.3048" layer="16"/>
+<wire x1="72.8" y1="33" x2="69.905" y2="33" width="0.3048" layer="16"/>
 <wire x1="69.905" y1="33" x2="69.87" y2="33.035" width="0.1524" layer="16"/>
 </signal>
@@
 <contactref element="U2" pad="1"/>
 <contactref element="U$2" pad="1"/>
-<wire x1="75.5" y1="35.6" x2="71.165" y2="35.6" width="0.1524" layer="16"/>
-<wire x1="71.165" y1="35.6" x2="69.87" y2="34.305" width="0.1524" layer="16"/>
+<wire x1="75.5" y1="35.6" x2="71.165" y2="35.6" width="0.3048" layer="16"/>
+<wire x1="71.165" y1="35.6" x2="69.87" y2="34.305" width="0.3048" layer="16"/>
 </signal>
 <signal name="N$33">
@@
 <wire x1="64.93" y1="28.57" x2="64.93" y2="30.495" width="0.3048" layer="16"/>
 </signal>
-<signal name="VIN-">
-<contactref element="U2" pad="7"/>
-<contactref element="R3" pad="2"/>
-<wire x1="64.93" y1="33.035" x2="60.465" y2="33.035" width="0.508" layer="16"/>
-<wire x1="60.465" y1="33.035" x2="59.4" y2="34.1" width="0.508" layer="16"/>
-<wire x1="59.4" y1="34.1" x2="59.4" y2="34.5" width="0.1524" layer="16"/>
-</signal>
 </signals>
