File: hardware/Eagle Designs/Solar Panel Board/Solar Panel Board v2.sch (EAGLE design)
At the start: 44 parts, among them J1 MOLEX_503763-0291MOLEX_503763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, J2 MOLEX_503763-0491MOLEX_503763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, J3 MOLEX_503763-0291MOLEX_503763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, U1 TMP36GSZ, U2 INA219BIDR

Commit message: Updated BOMs and edited Solar Panel Board v2
Parts:
- C1: value (none) -> 0.1uF
Changed lines of the file:
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@@
 <part name="U1" library="TMP36GSZ" deviceset="TMP36GSZ" device=""/>
 <part name="J3" library="Molex - 503763-0291" deviceset="MOLEX_503763-0291" device="MOLEX_503763-0291_0_0"/>
-<part name="C1" library="HSFL_Main_Library" deviceset="CAP" device="0805"/>
+<part name="C1" library="HSFL_Main_Library" deviceset="CAP" device="0805" value="0.1uF"/>
 <part name="U2" library="INA219BIDR" deviceset="INA219BIDR" device=""/>
 <part name="C2" library="HSFL_Main_Library" deviceset="CAP" device="0805" value="0.1uF"/>

Commit message: Add files via upload
Edited Solar Panel Board v2
Connections:
- removed net VIN-: R3.2, U2.VIN-
- net GND: now also R3.2, U2.VIN-
Changed lines of the file:
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@@
 <label x="398.78" y="-17.78" size="1.778" layer="95"/>
+</segment>
+<segment>
+<pinref part="U2" gate="A" pin="VIN-"/>
+<wire x1="355.6" y1="-7.62" x2="353.06" y2="-7.62" width="0.1524" layer="91"/>
+<pinref part="R3" gate="G$1" pin="2"/>
+<label x="355.6" y="-10.16" size="1.778" layer="95"/>
 </segment>
 </net>
@@
 </segment>
 </net>
-<net name="VIN-" class="0">
-<segment>
-<pinref part="U2" gate="A" pin="VIN-"/>
-<wire x1="355.6" y1="-7.62" x2="353.06" y2="-7.62" width="0.1524" layer="91"/>
-<pinref part="R3" gate="G$1" pin="2"/>
-<label x="355.6" y="-10.16" size="1.778" layer="95"/>
-</segment>
-</net>
