File: hardware/Eagle Designs/Solar Panel Board/Solar Panel Board v7.0.sch (EAGLE design)
At the start: 35 parts, among them J1 M55-6021242R, U1 TMP36GSZ

Commit message: Updated Artemis v2 EAGLE library, solar panel board, and antenna board
Connections:
- net GND: now also J1.GND; no longer J1.P$1, J1.P$2, J1.P$3, J1.P$4
Changed lines of the file:
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@@
 <attribute name="NAME" x="518.28" y="-33.52" size="1.778" layer="95" rot="R270"/>
 </instance>
-<instance part="J1" gate="G$1" x="386.08" y="-35.56" smashed="yes">
-<attribute name="NAME" x="378.46" y="-22.479" size="1.778" layer="95"/>
-<attribute name="VALUE" x="378.46" y="-50.292" size="1.778" layer="96"/>
+<instance part="J1" gate="G$1" x="383.54" y="-30.48" smashed="yes">
+<attribute name="NAME" x="375.92" y="-19.939" size="1.778" layer="95"/>
+<attribute name="VALUE" x="375.92" y="-22.352" size="1.778" layer="96"/>
 </instance>
 </instances>
@@
 </segment>
 <segment>
-<wire x1="396.24" y1="-30.48" x2="398.78" y2="-30.48" width="0.1524" layer="91"/>
-<label x="398.78" y="-30.48" size="1.778" layer="95"/>
+<wire x1="391.16" y1="-30.48" x2="393.7" y2="-30.48" width="0.1524" layer="91"/>
+<label x="393.7" y="-30.48" size="1.778" layer="95"/>
 <pinref part="J1" gate="G$1" pin="6"/>
 </segment>
@@
 </segment>
 <segment>
-<pinref part="J1" gate="G$1" pin="P$1"/>
-<wire x1="375.92" y1="-43.18" x2="373.38" y2="-43.18" width="0.1524" layer="91"/>
-<label x="373.38" y="-43.18" size="1.778" layer="95"/>
-</segment>
-<segment>
-<pinref part="J1" gate="G$1" pin="P$3"/>
-<wire x1="375.92" y1="-45.72" x2="373.38" y2="-45.72" width="0.1524" layer="91"/>
-<label x="373.38" y="-45.72" size="1.778" layer="95"/>
-</segment>
-<segment>
-<pinref part="J1" gate="G$1" pin="P$2"/>
-<wire x1="396.24" y1="-43.18" x2="398.78" y2="-43.18" width="0.1524" layer="91"/>
-<label x="398.78" y="-43.18" size="1.778" layer="95"/>
-</segment>
-<segment>
-<pinref part="J1" gate="G$1" pin="P$4"/>
-<wire x1="396.24" y1="-45.72" x2="398.78" y2="-45.72" width="0.1524" layer="91"/>
-<label x="398.78" y="-45.72" size="1.778" layer="95"/>
-</segment>
-<segment>
 <wire x1="375.92" y1="-27.94" x2="373.38" y2="-27.94" width="0.1524" layer="91"/>
 <label x="373.38" y="-27.94" size="1.778" layer="95" rot="MR0"/>
@@
 </segment>
 <segment>
-<wire x1="396.24" y1="-27.94" x2="398.78" y2="-27.94" width="0.1524" layer="91"/>
-<label x="398.78" y="-27.94" size="1.778" layer="95"/>
+<wire x1="391.16" y1="-27.94" x2="393.7" y2="-27.94" width="0.1524" layer="91"/>
+<label x="393.7" y="-27.94" size="1.778" layer="95"/>
 <pinref part="J1" gate="G$1" pin="4"/>
+</segment>
+<segment>
+<pinref part="J1" gate="G$1" pin="GND"/>
+<wire x1="383.54" y1="-43.18" x2="383.54" y2="-45.72" width="0.1524" layer="91"/>
+<label x="383.54" y="-45.72" size="1.778" layer="95" rot="MR180"/>
 </segment>
 </net>
 <net name="N$1" class="0">
 <segment>
-<pinref part="J1" gate="G$1" pin="7"/>
 <wire x1="375.92" y1="-33.02" x2="373.38" y2="-33.02" width="0.1524" layer="91"/>
 <label x="373.38" y="-33.02" size="1.778" layer="95" rot="MR0"/>
+<pinref part="J1" gate="G$1" pin="7"/>
 </segment>
 <segment>
+<wire x1="391.16" y1="-33.02" x2="393.7" y2="-33.02" width="0.1524" layer="91"/>
+<label x="393.7" y="-33.02" size="1.778" layer="95"/>
 <pinref part="J1" gate="G$1" pin="8"/>
-<wire x1="396.24" y1="-33.02" x2="398.78" y2="-33.02" width="0.1524" layer="91"/>
-<label x="398.78" y="-33.02" size="1.778" layer="95"/>
 </segment>
 </net>
@@
 </segment>
 <segment>
-<wire x1="396.24" y1="-25.4" x2="398.78" y2="-25.4" width="0.1524" layer="91"/>
-<label x="398.78" y="-25.4" size="1.778" layer="95"/>
+<wire x1="391.16" y1="-25.4" x2="393.7" y2="-25.4" width="0.1524" layer="91"/>
+<label x="393.7" y="-25.4" size="1.778" layer="95"/>
 <pinref part="J1" gate="G$1" pin="2"/>
 </segment>
