File: hardware/Eagle Designs/BBB_OBC v2/On Board Computer.brd (EAGLE design)
At the start: 90.2 x 95.5 mm, 25 parts, among them J1 MOLEX_503763-0491MOLEX_503763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, J10 503763-0591, J11 503763-0591, J12 503763-0691, J13 MOLEX_503763-0291MOLEX_503763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, J14 MOLEX_503763-0491MOLEX_503763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, J15 MOLEX_503763-0491MOLEX_503763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, J2 MOLEX_503763-0491MOLEX_503763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, J3 503763-0591, J4 503763-0591, J5 MOLEX_503763-0491MOLEX_503763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, J6 MOLEX_503763-0491MOLEX_503763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, J7 MOLEX_503763-0491MOLEX_503763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, J8 503763-0691, J9 MOLEX_503763-0491MOLEX_503763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, P8 SSW-123-02-G-D, P9 SSW-123-02-G-D, U1 ADT7311, U2 TMUX1108PWR, U3 AD7887ARMZ-REEL

Commit message: Uploaded OBC version 2
Parts:
- removed J9: MOLEX_503763-0491MOLEX_503763-0491_0_0, Molex - 503763-0491:MOLEX_503763-0491_0
- added C2, C3: 1uF, HSFL_Main_Library:0805
- added JP1: MOLEX_503763-0491MOLEX_503763-0491_0_0, Molex - 503763-0491:MOLEX_503763-0491_0
- added JP5: MOLEX_503763-0291MOLEX_503763-0291_0_0, Molex - 503763-0291:MOLEX_503763-0291_0
- added JP6, JP7: 503763-0691, Improved Molex 503763-0691:CONN_503763-0691_MOL
- added U4: LTC1477CS8LINEAR_TECHNOLOGY_LTC1477CS8_0_2, Artemis:LINEAR_TECHNOLOGY_LTC1477CS8_2
- added X1: C25582-40G-M36-0A, Adafruit - C25582-40G-M36-0A:ADAFRUIT_C25582-40G-M36-0A_0
- added X2: SSW-120-02-G-D, con-samtec:SSW-120-02-G-D
- J10, J11: device Molex - 503763-0591:CONN_5037630591_MOL -> Improved Molex 503763-0591:CONN_5037630591_MOL
- J12, J8: device Molex - 503763-0691:CONN_503763-0691_MOL -> Improved Molex 503763-0691:CONN_503763-0691_MOL
- J3, J4: value 503763-0591 -> MOLEX_503763-0491MOLEX_503763-0491_0_0; device Molex - 503763-0591:CONN_5037630591_MOL -> Molex - 503763-0491:MOLEX_503763-0491_0
- moved J8 27.4 mm to (30.4, 8.20), flipped to the bottom, turned to 180 degrees
- moved J6 27.4 mm to (8.60, 79.6), flipped to the bottom, turned to 270 degrees
- moved U2 27.3 mm to (36.7, 55.1), flipped to the bottom, turned to 180 degrees
- moved J10 22.3 mm to (29.2, 27.6), flipped to the bottom, turned to 90 degrees
- moved J4 17.8 mm to (82.2, 29.2), flipped to the bottom, turned to 90 degrees
- moved J3 17.3 mm to (75.0, 29.2), flipped to the bottom, turned to 270 degrees
- moved J12 15.8 mm to (46.4, 8.00), flipped to the bottom, turned to 180 degrees
- moved J11 14.2 mm to (16.4, 8.20), flipped to the bottom
- moved J7 12.2 mm to (11.2, 28.2), flipped to the bottom, turned to 270 degrees
- moved J2 9.62 mm to (74.8, 40.6), flipped to the bottom, turned to 270 degrees
- moved J1 9.62 mm to (82.2, 40.6), flipped to the bottom, turned to 90 degrees
- moved J15 6.00 mm to (74.4, 8.00), flipped to the bottom
- moved U1 5.83 mm to (48.9, 54.8), flipped to the bottom
- moved J14 4.60 mm to (61.0, 8.00), flipped to the bottom
- moved J13 3.40 mm to (85.0, 77.6), flipped to the bottom, turned to 90 degrees
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Connections:
- removed net ID_MICRO: J3.4, J4.2
- removed net ID_RP: H1.1.17
- new net GPIO12: X1.32
- new net GPIO13: X1.33
- new net GPIO16: X1.36
- new net GPIO17: JP6.1, X1.11
- new net GPIO19: X1.35
- new net GPIO20: X1.38
- new net GPIO21: X1.40
- new net GPIO22: JP6.4, X1.15
- new net GPIO23: JP6.3, X1.16
- new net GPIO24: JP6.5, X1.18
- new net GPIO25: JP6.6, X1.22
- new net GPIO26: X1.37
- new net GPIO27: JP6.2, X1.13
- new net GPIO6: X1.31
- new net RPI_5V_PWR_IN: C2.1, U4.1, U4.8, X1.2
- new net RPI_ENABLE: P8.7, U4.4
- new net SCL1_I2C: JP5.2, X1.5
- new net SDA1_I2C: JP5.1, X1.3
- new net SPI0_CE0_N: JP7.3, X1.24
- new net SPI0_CE1_N: JP7.5, X1.26
- new net SPI0_MISO: JP7.2, X1.21
- new net SPI0_MOSI: JP7.1, X1.19
- new net SPI0_SCLK: JP7.4, X1.23
- new net UART4_RXD: H1.1.1, P9.11
- new net UART4_TXD: H1.1.2, P9.13
- net +3V3_VCC: now also X1.1
- net 5V_SW1: now also C3.1, U4.2, U4.3, U4.6, U4.7
- net AGND: now also J7.1; no longer J7.4
- net ANI4: now also J7.2; no longer J7.3
- net ANI5: now also J7.3; no longer J7.2
- net ANI6: now also J7.4; no longer J7.1
- net D+_HOST: now also JP1.2; no longer H1.1.19, J6.2
- net D+_MICRO: now also J4.3; no longer J4.4
- net D-_HOST: now also JP1.3; no longer H1.1.20, J6.3
- net D-_MICRO: now also J4.2; no longer J4.3
- net GND: now also C2.2, C3.2, J10.6, J10.7, J11.6, J11.7, J12.7, J12.8, J3.4, J6.3, J8.7, J8.8, JP1.4, JP1.5, JP1.6, JP5.3, JP5.4, JP6.7, JP6.8, JP7.6, JP7.7, JP7.8, U4.5, X1.39; no longer J3.5, J9.1, J9.2, J9.5, J9.6
- net GPIO1_0: now also J12.1; no longer J12.3
- net GPIO1_1: now also J12.4; no longer J12.2
- net GPIO1_29: now also J12.5; no longer J12.4
- net GPIO1_4: now also J12.2; no longer J12.1
- net GPIO2_10: now also J10.1; no longer J10.5
- net GPIO2_22: now also J12.3; no longer J12.5
- net GPIO2_6: now also J10.5; no longer J10.1
- net GPIO2_7: now also J10.4; no longer J10.2
- net GPIO2_9: now also J10.2; no longer J10.4
- net S1: now also J14.1; no longer J14.4
- net S2: now also J14.2; no longer J14.3
- net S3: now also J14.3; no longer J14.2
- net S4: now also J14.4; no longer J14.1
- net UART1_RXD: now also J6.1; no longer J9.4
- net UART1_TXD: now also J6.2; no longer J9.3
- net UART2_RXD: now also X1.8; no longer H1.1.1
- net UART2_TXD: now also X1.10; no longer H1.1.2
- net VCC_HOST: now also JP1.1; no longer H1.1.18, J6.1
- net VCC_MICRO: now also J4.4; no longer J4.5
Routing:
- net VCC_HOST: track 168.6 -> 52.3 mm, vias 3 -> 1
- net D-_HOST: track 170.3 -> 55.2 mm, vias 3 -> 1
- net D+_HOST: track 166.6 -> 53.8 mm, vias 3 -> 1
- net GPIO23: track 0.00 -> 96.9 mm
- net GPIO22: track 0.00 -> 96.4 mm
- net 5V_SW1: track 67.1 -> 153.1 mm, vias 0 -> 2
- net GPIO24: track 0.00 -> 81.1 mm
- net GPIO17: track 0.00 -> 78.0 mm, vias 0 -> 2
- net RPI_5V_PWR_IN: track 0.00 -> 70.5 mm, vias 0 -> 2
- net +3V3_VCC: track 16.0 -> 84.2 mm, vias 0 -> 2
- net UART4_RXD: track 0.00 -> 67.5 mm
- net GPIO25: track 0.00 -> 66.1 mm
- net GPIO27: track 0.00 -> 58.1 mm, vias 0 -> 2
- net UART4_TXD: track 0.00 -> 56.6 mm
- net SPI0_CE0_N: track 0.00 -> 51.5 mm
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- added copper zone on layer 15, net GND
- added copper zone on layer 2, net GND
Other:
- board text added: "RPI Zero Camera"
- board text added: "Raspberry Pi Zero"
