File: hardware/Eagle Designs/BBB_OBC v2/On Board Computer.sch (EAGLE design)
At the start: 25 parts, among them J1 MOLEX_503763-0491MOLEX_503763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, J10 503763-0591, J11 503763-0591, J12 503763-0691, J13 MOLEX_503763-0291MOLEX_503763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, J14 MOLEX_503763-0491MOLEX_503763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, J15 MOLEX_503763-0491MOLEX_503763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, J2 MOLEX_503763-0491MOLEX_503763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, J3 503763-0591, J4 503763-0591, J5 MOLEX_503763-0491MOLEX_503763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, J6 MOLEX_503763-0491MOLEX_503763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, J7 MOLEX_503763-0491MOLEX_503763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, J8 503763-0691, J9 MOLEX_503763-0491MOLEX_503763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, P8 SSW-123-02-G-D, P9 SSW-123-02-G-D, U1 ADT7311, U2 TMUX1108PWR, U3 AD7887ARMZ-REEL

Commit message: Uploaded OBC version 2
Parts:
- removed J9: MOLEX_503763-0491MOLEX_503763-0491_0_0, Molex - 503763-0491:MOLEX_503763-0491MOLEX_503763-0491_0_0
- added C2, C3: 1uF, HSFL_Main_Library:CAP0805
- added JP1: MOLEX_503763-0491MOLEX_503763-0491_0_0, Molex - 503763-0491:MOLEX_503763-0491MOLEX_503763-0491_0_0
- added JP5: MOLEX_503763-0291MOLEX_503763-0291_0_0, Molex - 503763-0291:MOLEX_503763-0291MOLEX_503763-0291_0_0
- added JP6, JP7: 503763-0691, Improved Molex 503763-0691:503763-0691
- added U4: LTC1477CS8LINEAR_TECHNOLOGY_LTC1477CS8_0_2, Artemis:LTC1477CS8LINEAR_TECHNOLOGY_LTC1477CS8_0_2
- added X1: C25582-40G-M36-0A, Adafruit - C25582-40G-M36-0A:C25582-40G-M36-0A
- added X2: SSW-120-02-G-D, con-samtec:SSW-120-02-G-D
- J10, J11: device Molex - 503763-0591:503763-0591 -> Improved Molex 503763-0591:503763-0591
- J12, J8: device Molex - 503763-0691:503763-0691 -> Improved Molex 503763-0691:503763-0691
- J3, J4: value 503763-0591 -> MOLEX_503763-0491MOLEX_503763-0491_0_0; device Molex - 503763-0591:503763-0591 -> Molex - 503763-0491:MOLEX_503763-0491MOLEX_503763-0491_0_0
Connections:
- removed net ID_MICRO: J3.4, J4.2
- removed net ID_RP: H1.1.17
- new net GPIO12: X1.P$32
- new net GPIO13: X1.P$33
- new net GPIO16: X1.P$36
- new net GPIO17: JP6.1, X1.P$11
- new net GPIO19: X1.P$35
- new net GPIO20: X1.P$38
- new net GPIO21: X1.P$40
- new net GPIO22: JP6.4, X1.P$15
- new net GPIO23: JP6.3, X1.P$16
- new net GPIO24: JP6.5, X1.P$18
- new net GPIO25: JP6.6, X1.P$22
- new net GPIO26: X1.P$37
- new net GPIO27: JP6.2, X1.P$13
- new net GPIO6: X1.P$31
- new net RPI_5V_PWR_IN: C2.1, U4.1_VOUT, U4.2_VOUT, X1.P$2
- new net RPI_ENABLE: P8-7.1, U4.EN
- new net SCL1_I2C: JP5.2, X1.P$5
- new net SDA1_I2C: JP5.1, X1.P$3
- new net SPI0_CE0_N: JP7.3, X1.P$24
- new net SPI0_CE1_N: JP7.5, X1.P$26
- new net SPI0_MISO: JP7.2, X1.P$21
- new net SPI0_MOSI: JP7.1, X1.P$19
- new net SPI0_SCLK: JP7.4, X1.P$23
- new net UART4_RXD: H1.1.1, P9-11.1
- new net UART4_TXD: H1.1.2, P9-13.1
- net +3V3_VCC: now also X1.P$1
- net 5V_SW1: now also C3.1, U4.VIN1, U4.VIN2, U4.VIN3, U4.VINS
- net AGND: now also J7.1; no longer J7.4
- net ANI4: now also J7.2; no longer J7.3
- net ANI5: now also J7.3; no longer J7.2
- net ANI6: now also J7.4; no longer J7.1
- net D+_HOST: now also JP1.2; no longer H1.1.19, J6.2
- net D+_MICRO: now also J4.3; no longer J4.4
- net D-_HOST: now also JP1.3; no longer H1.1.20, J6.3
- net D-_MICRO: now also J4.2; no longer J4.3
- net GND: now also C2.2, C3.2, J10.PAD1, J10.PAD2, J11.PAD1, J11.PAD2, J12.PAD1, J12.PAD2, J3.4, J6.3, J8.PAD1, J8.PAD2, JP1.4, JP1.MNT_1, JP1.MNT_2, JP5.MNT_1, JP5.MNT_2, JP6.PAD1, JP6.PAD2, JP7.6, JP7.PAD1, JP7.PAD2, U4.GND, X1.P$39; no longer J3.5, J9.1, J9.2, J9.MNT_1, J9.MNT_2
- net GPIO1_0: now also J12.1; no longer J12.3
- net GPIO1_1: now also J12.4; no longer J12.2
- net GPIO1_29: now also J12.5; no longer J12.4
- net GPIO1_4: now also J12.2; no longer J12.1
- net GPIO2_10: now also J10.1; no longer J10.5
- net GPIO2_22: now also J12.3; no longer J12.5
- net GPIO2_6: now also J10.5; no longer J10.1
- net GPIO2_7: now also J10.4; no longer J10.2
- net GPIO2_9: now also J10.2; no longer J10.4
- net S1: now also J14.1; no longer J14.4
- net S2: now also J14.2; no longer J14.3
- net S3: now also J14.3; no longer J14.2
- net S4: now also J14.4; no longer J14.1
- net UART1_RXD: now also J6.1; no longer J9.4
- net UART1_TXD: now also J6.2; no longer J9.3
- net UART2_RXD: now also X1.P$8; no longer H1.1.1
- net UART2_TXD: now also X1.P$10; no longer H1.1.2
- net VCC_HOST: now also JP1.1; no longer H1.1.18, J6.1
- net VCC_MICRO: now also J4.4; no longer J4.5
