File: hardware/Eagle Designs/BBB_OBC v3/On Board Computer.sch (EAGLE design)
At the start: 33 parts, among them J1 MOLEX_503763-0491MOLEX_503763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, J10 503763-0591, J11 503763-0591, J12 503763-0691, J13 MOLEX_503763-0291MOLEX_503763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, J14 MOLEX_503763-0491MOLEX_503763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, J15 MOLEX_503763-0491MOLEX_503763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, J2 MOLEX_503763-0491MOLEX_503763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, J3 MOLEX_503763-0491MOLEX_503763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, J4 MOLEX_503763-0491MOLEX_503763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, J5 MOLEX_503763-0491MOLEX_503763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, J6 MOLEX_503763-0491MOLEX_503763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, J7 MOLEX_503763-0491MOLEX_503763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, J8 503763-0691, P8 SSW-123-02-G-D, P9 SSW-123-02-G-D, U1 ADT7311, U2 TMUX1108PWR, U3 AD7887ARMZ-REEL, U4 LTC1477CS8LINEAR_TECHNOLOGY_L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, X1 C25582-40G-M36-0A, X2 SSW-120-02-G-D

Commit message: OBC version 3 is finally here
Parts:
- removed J14, J15, J4, J5, JP1: MOLEX_503763-0491MOLEX_503763-0491_0_0, Molex - 503763-0491:MOLEX_503763-0491MOLEX_503763-0491_0_0
- removed J8: 503763-0691, Improved Molex 503763-0691:503763-0691
- removed R3: 10K, HSFL_Main_Library:RESISTOR0805-RES
- removed U3: AD7887ARMZ-REEL, Personal:AD7887ARMZ-REEL
- removed U4: LTC1477CS8LINEAR_TECHNOLOGY_LTC1477CS8_0_2, Artemis:LTC1477CS8LINEAR_TECHNOLOGY_LTC1477CS8_0_2
- added 3V3_BUS, GPS_BOOTSEL: (no value), wirepad:1,6/0,9
- added D1: (no value), led:LEDCHIP-LED0603
- added GND: GND, wirepad:1,6/0,9
- added J16, J9: U.FL-R-SMT-1(01), U.FL-R-SMT:U.FL-R-SMT-1(01)
- added JP4: (no value), microbuilder:HEADER-1X670MIL
- added R1: 27k, HSFL_Main_Library:RESISTOR0805-RES
- added U5: RFM69HCW, Artemis:RFM69HCW
- added U6: ORION_A38LORION_A38L, Artemis:ORION_A38LORION_A38L
- C1: value 0.1uF -> .1uF
- J3: value MOLEX_503763-0491MOLEX_503763-0491_0_0 -> MOLEX_503763-0291MOLEX_503763-0291_0_0; device Molex - 503763-0491:MOLEX_503763-0491MOLEX_503763-0491_0_0 -> Molex - 503763-0291:MOLEX_503763-0291MOLEX_503763-0291_0_0
- R2: value 10K -> 10k
- U1: value ADT7311 -> TMP36FSZR_8_ADI-L; device HSFL_Main_Library:ADT7311 -> TMP36FSZR_8:TMP36FSZR_8_ADI-L
- U2: value TMUX1108PWR -> LTC1477CS8LINEAR_TECHNOLOGY_LTC1477CS8_0_2; device SamacSys_Parts:TMUX1108PWR -> Artemis:LTC1477CS8LINEAR_TECHNOLOGY_LTC1477CS8_0_2
Connections:
- net ANI1 renamed AIN1
- net ANI3 renamed AIN3
- net ANI4 renamed AIN4
- net ANI5 renamed AIN5
- net ANI6 renamed AIN6
- removed net 5V_SW1: C3.1, H1.2.8, J13.1, U4.VIN1, U4.VIN2, U4.VIN3, U4.VINS
- removed net ANI0: H1.1.3, P9-39.1
- removed net ANI2: H1.1.5, P9-37.1
- removed net D: U2.D, U3.AIN0
- removed net D+_HOST: J5.3, JP1.2
- removed net D+_MICRO: J3.2, J4.3
- removed net D-_HOST: J5.2, JP1.3
- removed net D-_MICRO: J3.3, J4.2
- removed net GPIO12: X1.P$32
- removed net GPIO13: X1.P$33
- removed net GPIO16: X1.P$36
- removed net GPIO19: X1.P$35
- removed net GPIO20: X1.P$38
- removed net GPIO21: X1.P$40
- removed net GPIO26: X1.P$37
- removed net GPIO6: X1.P$31
- removed net GPIO_FAULT1: H1.1.40
- removed net GPIO_FAULT2: H1.1.46
- removed net GPIO_SLEEP1: H1.1.42
- removed net GPIO_SLEEP2: H1.1.48
- removed net GPIO_TRQ1: H1.1.38
- removed net GPIO_TRQ2: H1.1.44
- removed net I2C1_SCL: H1.1.43, P9-17.1
- removed net I2C1_SDA: H1.1.41, P9-18.1
- removed net S1: J14.1, U2.S1
- removed net S2: J14.2, U2.S2
- removed net S3: J14.3, U2.S3
- removed net S4: J14.4, U2.S4
- removed net S5: J15.4, U2.S5
- removed net S6: J15.3, U2.S6
- removed net S7: J15.2, U2.S7
- removed net S8: J15.1, U2.S8
- removed net U11_CT: R2.1, U1.CT
- removed net U11_INT: R3.1, U1.INT
- removed net UART4_RXD: H1.1.1, P9-11.1
- removed net UART4_TXD: H1.1.2, P9-13.1
- removed net VCC_HOST: J5.4, JP1.1
- removed net VCC_MICRO: J3.1, J4.4
- new net 3V3_BUS: 3V3_BUS.P, H1.2.27, H1.2.28, U6.GPS_CONST_PWR
- new net 5V_BUS: H1.2.25, H1.2.26
- new net AIN0: H1.1.3, P9-39.1, R1.1, R2.2
- new net AIN2: H1.1.5, J3.1, P9-37.1
- new net BUS_UART4_RXD(BBB_TX): H1.1.1, P9-13.1
- new net BUS_UART4_TXD(BBB_RX): H1.1.2, P9-11.1
- new net GPIO_10: P8-31.1
- new net GPS_BOOTSEL: GPS_BOOTSEL.P, U6.GPS_BOOTSEL
- new net GPS_RSTN: P8-32.1, U6.RSTN
- new net INTM: JP4.6
- new net N$17: J9.3, U6.GPS_ANT
- new net N$19: J16.3, U5.ANT
- new net N$21: D1.A, U6.GPS_LED
- new net RADIO_RESET: P8-36.1, U5.RESET
- new net SPI1_CS1: P9-42.1, U5.NSS
- new net SW_5V_1: H1.2.13, J13.1
- net +3V3_VCC: now also JP4.2, U1.!SHUTDOWN, U1.+VS, U5.3.3V, U6.GPS_3V3; no longer R2.2, R3.2, U1.VDD, X1.P$1
- net +5V_VCC: now also C3.1, U2.VIN1, U2.VIN2, U2.VIN3, U2.VINS; no longer U2.VDD, U3.VDD
- net GND: now also D1.C, GND.P, J16.1, J16.2, J3.2, J3.MNT_1, J3.MNT_2, J9.1, J9.2, JP4.3, R2.1, U5.GND, U6.2ND_GND, U6.GND, U6.GND_RF; no longer J14.MNT_1, J14.MNT_2, J15.MNT_1, J15.MNT_2, J3.4, J4.1, J5.1, J5.MNT_1, J5.MNT_2, J8.1, J8.2, J8.PAD1, J8.PAD2, JP1.4, JP1.MNT_1, JP1.MNT_2, U3.GND, U4.GND
- net GPIO1_16: no longer U2.A2
- net GPIO1_17: no longer U2.A0
- net GPIO1_28: no longer U2.A1
- net GPIO2_11: now also J11.5; no longer J11.1
- net GPIO2_12: now also J11.3; no longer J11.2
- net GPIO2_13: now also J11.4; no longer J11.3
- net GPIO2_23: now also J11.1; no longer J11.4
- net GPIO2_25: now also J11.2; no longer J11.5
- net GPIO3_21: no longer U2.EN
- net I2C2_SCL: now also JP4.4; no longer J8.3
- net I2C2_SDA: now also JP4.5; no longer J8.4
- net N$15: now also R1.2, U1.VOUT; no longer U2.VSS
- net RPI_5V_PWR_IN: now also U2.1_VOUT, U2.2_VOUT; no longer U4.1_VOUT, U4.2_VOUT
- net RPI_ENABLE: now also U2.EN; no longer U4.EN
- net SPI1_CS0: no longer H1.1.10, U1.CS, U3.CS
- net SPI1_D0: now also U5.MISO; no longer H1.1.11, U1.DOUT, U3.DOUT
- net SPI1_D1: now also U5.MOSI; no longer H1.1.12, U1.DIN, U3.DIN
- net SPI1_SCLK: now also U5.SCK; no longer H1.1.9, U1.SCLK, U3.SCLK
- net UART5_RXD: now also U6.GPS_TXD0; no longer J8.6
- net UART5_TXD: now also U6.GPS_RXDO; no longer J8.5
Other:
- note added: "BB TEMP SENSOR"
- note added: "Beaglebone Black"
- note added: "Modular IMU"
- note added: "Modular Radio"
- note added: "OBC TEMP SENSOR"
- note added: "Orion GPS Unit"
- note added: "PDU TEMP SENSOR"
- note added: "Raspberry Pi"
- note added: "Raspberry Pi Enable"
- note added: "Temp Sensor"
