File: hardware/Eagle Designs/PDU_v2/PDU_v2.brd (EAGLE design)
At the start: 160 x 100 mm, 163 parts, among them J1 5037630291, J10 5037630291, J11 5037630291, J12 5037630291, J13 5037630291, J14 5037630291, J15 5037630491, J16 5037630291, J17 5037630291, J18 5037630291, J19 5037630291, J2 5037630291, J3 5037630291, J4 5037630291, J5 5037630291, J6 5037630291, J7 5037630291, J8 5037630291, J9 5037630291, M1 BSZ100N06LS3, M2 BSZ100N06LS3, M3 BSZ033NE2LS5, M4 BSZ033NE2LS5, T1 2N5088, U1 DRV8847PWPR, U10 PE014006, U11 IRLML2803PBFCT-ND, U12 IRLML2803PBFCT-ND, U13 LT8390EFE#PBF, U14 ATSAMD51J19A-AU, U15 INA219BIDR, U2 DRV8847PWPR, U3 LTC1477CS8LINEAR_TECHNOLOGY_L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, U4 LTC1477CS8LINEAR_TECHNOLOGY_L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, U5 LTC1477CS8LINEAR_TECHNOLOGY_L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, U6 LTC1477CS8LINEAR_TECHNOLOGY_L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, U7 LTC1477CS8LINEAR_TECHNOLOGY_L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, U8 LTC1477CS8LINEAR_TECHNOLOGY_L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, U9 LTC1477CS8LINEAR_TECHNOLOGY_L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

Commit message: updated PDU v2 and Artemis Library
Parts:
- removed C30: (no value), HSFL_Main_Library:0805
- removed ISTHISTHERIGHTVALUE, ISTHISTHERIGHTVALUE1: 3.3k, HSFL_Main_Library:0805
- removed U$15, U$16: NDS8434, Artemis:SO08
- added C61, C64: 0.1 uF, HSFL_Main_Library:0805
- added C62, C63: 22 pF, HSFL_Main_Library:0805
- added C65: (no value), HSFL_Main_Library:0805
- added D2: 1655, Artemis:LED_1655
- added J20: 503182-1852, Artemis:MOLEX_503182-1852
- added J21: 5037630291, Artemis:CON_5037630291
- added J22: UJ31-CH-G1-SMT-TR, Artemis:CUI_UJ31-CH-G1-SMT-TR
- added R38, R41, R42: 10k, HSFL_Main_Library:0805
- added R39: 55k, HSFL_Main_Library:0805
- added R40: 100k, HSFL_Main_Library:0805
- added R43, R44: 3.3k, HSFL_Main_Library:0805
- added R48, R49: 5.1k, HSFL_Main_Library:0805
- added U$6, U$7: NDS8434, Artemis:SO08
- added Y1: ABS07-32.768KHZ-T, Artemis:XTAL_ABS07-32.768KHZ-T
- C54, C56: value (none) -> 10 uF
- C55, C57, C58: value (none) -> 1 uF
- C59, C60: value (none) -> 0.1 uF
- R37: value L_0805 -> 10 uH
Connections:
- net BUS_3V3_EN renamed BUS_3V3_EN1
- net BUS_5V_EN renamed BUS_5V_EN1
- net HB1_IN1 renamed IN1
- net HB1_IN2 renamed IN2
- net HB1_IN3 renamed IN3
- net HB1_IN4 renamed IN4
- net HB1_NSLEEP renamed SLEEP1
- net HB1_TRQ renamed TRQ1
- net HB2_IN1 renamed IN5
- net HB2_IN2 renamed IN6
- net HB2_IN3 renamed IN7
- net HB2_IN4 renamed IN8
- net HB2_NSLEEP renamed SLEEP2
- net HB2_TRQ renamed TRQ2
- net N$10 renamed BUS_3V3_TRSS
- net N$26 renamed BUS_5V_TRSS
- net N$30 renamed BUS_5V_FB
- net N$39 renamed SW_12V_IN1
- net N$43 renamed SW_12V_PGOOD
- net N$5 renamed SW_12V_EN1
- net N$51 renamed SW_12V_FB
- net N$9 renamed BUS_3V3_FB
- net NAMETHIS renamed +5V_BUS
- net PG_3V3_BUS renamed BUS_3V3_PG
- net PG_5V_BUS renamed BUS_5V_PG
- net SW_3V3_EN_1 renamed SW_3V3_EN1
- net SW_3V3_EN_2 renamed SW_3V3_EN2
- net SW_5V_EN_1 renamed SW_5V_EN1
- net SW_5V_EN_2 renamed SW_5V_EN2
- net SW_5V_EN_3 renamed SW_5V_EN3
- net SW_5V_EN_4 renamed SW_5V_EN4
- net SW_VBATT_EN renamed SW_VBATT_EN1
- removed net BURN_RELAY_A: R7.2, T1.2
- removed net ENAB_BURN1: R10.1, R9.2
- removed net ENAB_BURN2: R12.2, R13.1
- removed net HB1_FAULT: ISTHISTHERIGHTVALUE.1, U1.8
- removed net HB2_FAULT: ISTHISTHERIGHTVALUE1.1, U2.8
- removed net N$59: R34.2, U15.3
- removed net NAMETHIS__: ISTHISTHERIGHTVALUE.2, ISTHISTHERIGHTVALUE1.2
- new net +3V3: C64.1, D2.3, J20.4, J21.1, R38.2, R42.2
- new net +3V3_BUS: R43.1, R44.1
- new net 5V_BURN: R7.2, T1.2, U14.28
- new net BURN1_EN: R10.1, R9.2, U14.60
- new net BURN2_EN: R12.2, R13.1, U14.32
- new net CUS_SDA: R34.2, U14.25, U15.3
- new net FAULT1: R43.2, U1.8
- new net FAULT2: R44.2, U2.8
- new net N$54: C61.1, R39.1, R40.1, U14.15
- new net N$60: C62.2, U14.1, Y1.2
- new net N$62: C63.2, U14.2, Y1.1
- new net N$63: R39.2, R41.1
- new net N$64: R41.2
- new net N$65: D2.2, U14.42
- new net SPI1_CS0: J20.2, R42.1, U14.51
- new net SPI1_D0: J20.7, U14.31
- new net SPI1_D1: J20.3, U14.29
- new net SPI1_SCLK: J20.5, U14.30
- new net SWCLK: J21.3, U14.57
- new net SWDIO: J21.2, U14.58
- new net USB_CC1: J22.A5, R48.2
- new net USB_CC2: J22.B5, R49.2
- new net USB_D+: J22.A6, J22.B6, U14.46
- new net USB_D-: J22.A7, J22.B7, U14.45
- new net USB_VBUS: C65.2, J22.A4, J22.A9, J22.B4, J22.B9
- net 12V_OUT: now also C78.1, C79.1, C80.1, C81.1, D4.A, R4.2, R5.2, U13.15
- net GND: now also C61.2, C62.1, C63.1, C64.2, C65.1, D2.1, J20.6, J20.P1, J20.P2, J20.P3, J20.P4, J20.P5, J21.4, J22.A1, J22.A12, J22.B1, J22.B12, J22.SH1, J22.SH2, J22.SH3, J22.SH4, J22.SH5, J22.SH6, R38.1, R40.2, R48.1, R49.1
- net N$13: now also U$6.1, U$6.2, U$6.3, U$7.1, U$7.2, U$7.3; no longer U$15.1, U$15.2, U$15.3, U$16.1, U$16.2, U$16.3
- net N$15: now also U$7.4; no longer U$16.4
- net N$18: now also U$6.4; no longer U$15.4
- net VBURN1: now also U$6.5, U$6.6, U$6.7, U$6.8; no longer U$15.5, U$15.6, U$15.7, U$15.8
- net VBURN2: now also U$7.5, U$7.6, U$7.7, U$7.8; no longer U$16.5, U$16.6, U$16.7, U$16.8
- net VCC: no longer C78.1, C79.1, C80.1, C81.1, D4.A, R4.2, R5.2, U13.15

Commit message: updated PDU v2 Microprocessor schematic
Parts:
- added C30: 4.7 uF, HSFL_Main_Library:0805
- added C66: 47 nF, HSFL_Main_Library:0805
- added C67, C68: 10 uF, HSFL_Main_Library:0805
- added C69: 44 uF, HSFL_Main_Library:0805
- added C70, C71: 1 uF, HSFL_Main_Library:0805
- added L2: 1 uH, HSFL_Main_Library:ELL4GG
- added LED1: LED0805, HSFL_Main_Library:LED_0805
- added R45, R52, R54, R55, R56, R57: 10k, HSFL_Main_Library:0805
- added R50: 5.23k, HSFL_Main_Library:0805
- added R51: 30.1k, HSFL_Main_Library:0805
- added R53: 383, HSFL_Main_Library:0805
- added R58: 2k, HSFL_Main_Library:0805
- added SW1: KMR231GLFS, Artemis:KMR2XXG_CNK
- added U$8: BQ25883RGER, Artemis:QFN50P400X400X100-25N
- added U16: MAX706RESA+T, Artemis:21-0041B_8_MXM
- added U17: MAX16998AAUA+T, Artemis:21-0036K_MXM
- U14: value ATSAMD51J19A-AU -> ATSAME51N19A-AF; device Artemis:TQFP64_PT_MCH -> Artemis:TQFP100_14X14MC_MCH
- moved C64 2339.6 mm to (-331.5, 781.0)
- moved D2 2323.0 mm to (-330.2, 773.4)
- moved R40 2260.9 mm to (-331.5, 760.7)
- moved R41 2257.1 mm to (-331.5, 765.8)
- moved R39 2252.1 mm to (-331.5, 755.6)
- moved C63 2231.7 mm to (-326.4, 745.5)
- moved C62 2227.9 mm to (-331.5, 745.5)
- moved Y1 2215.3 mm to (-331.5, 739.1)
- moved C61 2212.7 mm to (-331.5, 750.6)
- moved R38 2186.1 mm to (-326.4, 729.0)
- moved C60 2182.5 mm to (-331.5, 729.0)
- moved C59 2173.5 mm to (-326.4, 723.9)
- moved C58 2169.8 mm to (-331.5, 723.9)
- moved C57 2160.8 mm to (-326.4, 718.8)
- moved C56 2157.1 mm to (-331.5, 718.8)
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Connections:
- new net 5V_BURN_RELAY: U14.54
- new net CUS_SCL: R36.2, U$8.5, U14.73, U15.4
- new net N$10: LED1.1, R45.2
- new net N$26: C30.1, U$8.11
- new net N$30: R53.2, U$8.8
- new net N$39: C66.1, U$8.12
- new net N$43: C67.1, L2.P$1, U$8.21, U$8.22
- new net N$5: R50.1, R51.2, R52.2, U$8.7
- new net N$51: C66.2, L2.P$2, U$8.17, U$8.18
- new net N$59: C61.1, R39.1, R40.1, U14.7
- new net N$9: LED1.2, U$8.2
- new net RESET: C71.1, R55.1, R56.1, R58.2, SW1.1, SW1.2, U14.88, U17.7
- new net SPI1_CT: U14.52
- new net SPI1_INT: U14.53
- new net USB_JUMP1: C69.1, U$8.15, U$8.16
- new net USB_JUMP_BAT: C68.1, U$8.13, U$8.14
- new net WDT_WDI: U16.6, U17.6
- net +3V3: now also R54.1, R55.2, R58.1, U16.2
- net 5V_BURN: no longer U14.28
- net BURN1_EN: now also U14.55; no longer U14.60
- net BURN2_EN: now also U14.70; no longer U14.32
- net BUS_3V3_EN1: now also U14.74
- net BUS_3V3_PG: now also U14.71
- net BUS_5V_EN1: now also U14.87
- net BUS_5V_PG: now also U14.75
- net CUS_SDA: now also U$8.4, U14.72; no longer U14.25
- net FAULT1: now also U14.65
- net FAULT2: now also U14.80
- net GND: now also C30.2, C67.2, C68.2, C69.2, C70.2, C71.2, R51.1, R52.1, R53.1, SW1.3, SW1.4, SW1.5, U$8.19, U$8.20, U$8.25, U14.11, U14.12, U14.24, U14.25, U14.30, U14.31, U14.38, U14.39, U14.50, U14.51, U14.62, U14.63, U14.76, U14.77, U14.90, U14.92, U16.3, U16.4, U17.5; no longer U14.21, U14.22, U14.33, U14.34, U14.47, U14.48, U14.54, U14.56, U14.7, U14.8
- net IN1: now also U14.34
- net IN2: now also U14.35
- net IN3: now also U14.36
- net IN4: now also U14.37
- net IN5: now also U14.67
- net IN6: now also U14.68
- net IN7: now also U14.69
- net IN8: now also U14.78
- net N$46: now also U14.91; no longer U14.55
- net N$54: now also R56.2, U16.7, U16.8; no longer C61.1, R39.1, R40.1, U14.15
- net N$58: now also U14.89; no longer U14.53
- net N$61: now also R57.2, U17.8; no longer R36.2, U15.4
- net N$65: now also U14.95; no longer U14.42
- net PCM_VBATT: now also R57.1, U17.1
- net SLEEP1: now also U14.64
- net SLEEP2: now also U14.79
- net SPI1_CS0: now also U14.49; no longer U14.51
- net SPI1_D0: now also U14.48; no longer U14.31
- net SPI1_D1: now also U14.46; no longer U14.29
- net SPI1_SCLK: now also U14.47; no longer U14.30
- net SWCLK: now also R54.2, U14.93; no longer U14.57
- net SWDIO: now also U14.94; no longer U14.58
- net SW_12V_EN1: now also U14.40
- net SW_12V_PGOOD: now also U14.41
- net SW_3V3_EN1: now also U14.42
- net SW_3V3_EN2: now also U14.43
- net SW_5V_EN1: now also U14.44
- net SW_5V_EN2: now also U14.45
- net SW_5V_EN3: now also U14.56
- net SW_5V_EN4: now also U14.57
- net SW_VBATT_EN1: now also U14.58
- net TRQ1: now also U14.66
- net TRQ2: now also U14.81
- net USB_D+: now also U$8.24, U14.86; no longer U14.46
- net USB_D-: now also U$8.1, U14.85; no longer U14.45
- net USB_VBUS: now also C70.1, R45.1, R50.2, U$8.23

Commit message: updated PDU v2
Parts:
- removed U$22: LT8609A, Artemis:MSOP_10PAD
- removed U$7: NDS8434, Artemis:SO08
- removed U$8: BQ25883RGER, Artemis:QFN50P400X400X100-25N
- added C100, C89, C98, C99: 4.7 uF, HSFL_Main_Library:0805
- added C72, C82, C91, C96: 0.1 uF, HSFL_Main_Library:0805
- added C73, C90, C94: 1 uF, HSFL_Main_Library:0805
- added C83: 0.01 uF, HSFL_Main_Library:0805
- added C84: 10pF, HSFL_Main_Library:0805
- added C85: 47uF, HSFL_Main_Library:1210
- added C86, C88: 4.7uF, HSFL_Main_Library:0805
- added C87: 0.1uF, HSFL_Main_Library:0805
- added C92: 33 pF, HSFL_Main_Library:0805
- added C93: 0 uF, HSFL_Main_Library:0805
- added C95, C97: 10 uF, HSFL_Main_Library:0805
- added CR1, CR2, CR3, CR4, CR5, CR6, CR7: PMEG10020ELRX, Artemis:CFP3_SOD123W_NEX
- added D3: SBR2A40P1Q-7, Artemis:POWERDI-123
- added J23, J24, J25: 2PIN_HEADER, HSFL_Main_Library:2MM_2PIN_HEADER
- added J26: 1729128, Artemis:CONN_1729128_PXC
- added L6: 10uH, HSFL_Main_Library:XFL4030472MEB
- added LED2, LED3: LED_0805, HSFL_Main_Library:LED_0805
- added R59: 80k, HSFL_Main_Library:0805
- added R60: 50k, HSFL_Main_Library:0805
- added R61, R62, R77, R82, R84: 10k, HSFL_Main_Library:0805
- added R63: 125k, HSFL_Main_Library:0805
- added R64, R72, R73, R74, R75: 1M, HSFL_Main_Library:0805
- added R65: 190k, HSFL_Main_Library:0805
- added R66: 9k, HSFL_Main_Library:0805
- added R67, R85: 15k, HSFL_Main_Library:0805
- added R68: 40.2K, HSFL_Main_Library:0805
- added R69: 100K, HSFL_Main_Library:0805
- added R70: 1.0M, HSFL_Main_Library:0805
- added R71: 69.8K, HSFL_Main_Library:0805
- added R76: 27.4k, HSFL_Main_Library:0805
- added R78, R81: 2k, HSFL_Main_Library:0805
- added R79: 71.5k, HSFL_Main_Library:0805
- added R80: 86.6k, HSFL_Main_Library:0805
- added R83: 40.2, HSFL_Main_Library:0805
- added R86, R87, R90: 1k, HSFL_Main_Library:0805
- added R88: 2.2 uH, Artemis:RESC0805X60N
- added R89: 100, HSFL_Main_Library:0805
- added U18: ADT7311WTRZ, Artemis:R_8_ADI
- added U19: NTGD1100LT1G, Artemis:TSOP6_1P70X3P10_ONS
- added U20: AO3400, Artemis:SOT-23-3L_AOS
- added U21, U22, U23: LT8609A, HSFL_Main_Library:MSOP-10_MSE
- C16: value 0.1 uF -> 0.1uF
- C17: value 1 uF -> 1uF
- C24, C36: value 22 uF -> 47 uF; device HSFL_Main_Library:1206 -> HSFL_Main_Library:0805
- C31: value 10 nF -> 0.01 uF
- J10: value 5037630291 -> 5037630691; device Artemis:CON_5037630291 -> Artemis:CONN_503763-0691_MOL
- J11, J12: value 5037630291 -> 2PIN_HEADER; device Artemis:CON_5037630291 -> HSFL_Main_Library:2MM_2PIN_HEADER
- J15: value 5037630491 -> 2PIN_HEADER; device Artemis:CON_5037630491 -> HSFL_Main_Library:2MM_2PIN_HEADER
- J7, J8, J9: value 5037630291 -> 5037630491; device Artemis:CON_5037630291 -> Artemis:CON_5037630491
- R15: value 309 K -> 300k
- R16, R24: value 100 K -> 49.9k
- R17: value 1 M -> 1M
- R23: value 187 K -> 182k
- U$3, U$5: value LT8609A -> NDS8434; device Artemis:MSOP_10PAD -> Artemis:SO08
- U$6: value NDS8434 -> BQ25883RGER; device Artemis:SO08 -> Artemis:QFN50P400X400X100-25N
- U8: value LTC1477CS8LINEAR_TECHNOLOGY_LTC1477CS8_0_2 -> LT8609A; device Artemis:LINEAR_TECHNOLOGY_LTC1477CS8_2 -> HSFL_Main_Library:MSOP-10_MSE
- moved R58 1912.6 mm to (-111.8, 193.0)
- moved R57 1908.1 mm to (-106.7, 193.0)
- moved R56 1897.4 mm to (-101.6, 193.0)
- moved R55 1875.3 mm to (-96.5, 193.0)
- moved R54 1872.2 mm to (-91.4, 193.0)
- moved C71 1869.0 mm to (-106.7, 182.9)
- moved U17 1861.5 mm to (-115.6, 152.4)
- moved SW1 1847.8 mm to (-82.5, 152.4)
- moved C70 1836.1 mm to (-101.6, 182.9)
- moved C69 1831.7 mm to (-96.5, 182.9)
- moved C68 1828.6 mm to (-91.4, 182.9)
- moved C67 1825.4 mm to (-86.4, 182.9)
- moved R53 1824.5 mm to (-86.4, 193.0)
- moved C66 1820.1 mm to (-81.3, 182.9)
- moved R52 1815.0 mm to (-81.3, 193.0)
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Connections:
- net N$59 renamed BATTERY_DC
- net SPI1_CT renamed UART2_RXD
- net SPI1_D0 renamed SPI_MISO
- net SPI1_D1 renamed SPI_MOSI
- net SPI1_INT renamed UART2_TXD
- net SPI1_SCLK renamed SPI_SCK
- removed net 3V3_SW1: J15.1
- removed net 5V_SW4: J15.2
- removed net AGND: U$1.10
- removed net BAT_IN: J16.1
- removed net BST: U$1.6
- removed net BUS_3V3_EN1: U$3.EN/UV, U14.74
- removed net BUS_5V_EN1: U$5.EN/UV, U14.87
- removed net PGND: U$1.5
- removed net SPI1_CS0: J20.2, R42.1, U14.49
- removed net SW_5V_4: C17.1, U8.1, U8.8
- removed net VH: U$1.3
- removed net V_BATT: C1.1, C2.1, C4.1, C47.1, C48.1, M1.P$5, M1.P$6, M1.P$7, M1.P$8, M1.P$9, R2.2, U13.7
- new net 12V_SW1: C84.2, C85.1, C86.1, J10.3, L6.2, R69.2, R70.2
- new net 5V_USB_CHRG: CR7.2, H1.1.32
- new net BC_OUT: C94.2, C95.2, H1.2.41, H1.2.42, H1.2.43, H1.2.44, U$1.3
- new net BC_VCC: R78.2, R81.1
- new net BST_3V3_BUS: C87.1, U8.1
- new net BURNWIREHERE________________________: H1.2.8
- new net BUS_EN: C83.1, R65.2, U14.74, U19.2, U19.3, U21.10, U22.10
- new net FB_3V3_BUS: C84.1, R70.1, R71.2, U8.6
- new net GNDA: C90.2, C91.2, C92.1, C93.1, R77.2, R79.2, R80.2, R83.1, R86.2, U$1.10, U$1.13, U$1.14, U$1.15, U$1.16, U$1.8
- new net KAPT_HEAT_IN: J26.1
- new net MID: U20.2
- new net N$100: C96.2, U$1.6
- new net N$101: U$1.22
- new net N$59: H1.P$1, R72.2
- new net N$66: C72.1, U17.3
- new net N$67: H1.P$2, R73.2
- new net N$68: C73.1, U17.4
- new net N$69: R63.1, R64.2, U19.4
- new net N$70: R59.2, R60.1, U17.2
- new net N$71: H1.P$3, R74.2
- new net N$72: CR1.2, J11.1
- new net N$73: CR2.2, J12.1
- new net N$74: R89.2, R90.2, U20.3
- new net N$75: CR3.2, J15.1
- new net N$76: H1.1.49
- new net N$77: H1.1.51
- new net N$78: CR4.2, J23.1
- new net N$79: CR5.2, J24.1
- new net N$80: CR6.2, J25.1
- new net N$81: J18.4
- new net N$82: J19.4
- new net N$83: J20.6
- new net N$84: R35.2, U15.7
- new net N$85: LED2.2, U$1.25
- new net N$86: LED2.1, R78.1
- new net N$87: C90.1, U$1.9
- new net N$88: R79.1, U$1.24
- new net N$89: R80.1, U$1.23
- new net N$90: C91.1, U$1.11
- new net N$91: LED3.2, U$1.26
- new net N$92: LED3.1, R81.2
- new net N$93: R82.2, R83.2, U$1.21
- new net N$94: R84.2, U$1.19
- new net N$95: C92.2, R82.1
- new net N$96: R84.1, R85.2, U$1.20
- new net N$97: C93.2, R85.1
- new net N$98: R89.1, U$1.12
- new net N$99: R86.1, R87.1, U$1.17
- new net PG_3V3_BUS: R69.1, U8.8
- new net R1/C1: C83.2, R63.2, U19.6
- new net RT_3V3_BUS: R68.2, U8.4
- new net SOLAR_VS: C29.1, U15.5
- new net SPI2_CS0: H1.1.10, U18.4
- new net SPI2_CT: R61.1, U18.6
- new net SPI2_D0: H1.1.11, U18.2
- new net SPI2_D1: H1.1.12, U18.3
- new net SPI2_INT: R62.1, U18.5
- new net SPI2_SCLK: H1.1.9, U18.1
- new net SPI_SD_CS: J20.1, R42.1, U14.49
- new net SW_3V3_BUS: C87.2, L6.1, U8.2
- new net TRSS_3V3_BUS: C16.1, U8.7
- new net VCC_3V3_BUS: C17.1, U8.3
- new net VLIM: R76.2, R77.1, U$1.18
- new net WDT_EN: R57.1, U17.8
- net +3V3: now also R60.2, R61.2, R62.2
- net 12V_OUT: now also C88.1, U8.9
- net BUS_3V3: now also C99.1, H1.2.27, H1.2.28
- net BUS_3V3_FB: now also U21.6; no longer U$3.FB
- net BUS_3V3_PG: now also U21.8; no longer U$3.PG
- net BUS_3V3_TRSS: now also U21.7; no longer U$3.TR/SS
- net BUS_5V: now also C100.1, C82.1, H1.2.25, H1.2.26, U18.8; no longer C16.1, U8.2, U8.3, U8.7
- net BUS_5V_FB: now also U22.6; no longer U$5.FB
- net BUS_5V_PG: now also U22.8; no longer U$5.PG
- net BUS_5V_TRSS: now also U22.7; no longer U$5.TR/SS
- net BUS_VBATT: now also C1.1, C2.1, C4.1, C47.1, C48.1, H1.2.45, H1.2.46, M1.P$5, M1.P$6, M1.P$7, M1.P$8, M1.P$9, R2.2, U13.7
- net CUS_SCL: now also H1.1.43, U$6.5; no longer U$8.5
- net CUS_SDA: now also H1.1.41, U$6.4; no longer U$8.4
- net FAULT1: now also H1.1.40
- net FAULT2: now also H1.1.46
- net GND: now also C100.2, C72.2, C73.2, C82.2, C85.2, C86.2, C88.2, C89.1, C94.1, C95.1, C97.1, C98.1, C99.2, D3.A, H1.2.14, H1.2.17, H1.2.21, H1.2.22, H1.2.29, H1.2.30, H1.2.32, H1.2.47, H1.2.48, H1.2.7, J10.5, J10.6, J11.2, J12.2, J15.2, J23.2, J24.2, J25.2, J26.2, J9.5, J9.6, R59.1, R65.1, R67.1, R68.1, R71.1, R72.1, R73.1, R74.1, R75.1, R90.1, U$1.5, U$6.19, U$6.20, U$6.25, U18.7, U19.1, U20.1, U21.11, U21.5, U22.11, U22.5, U23.11, U23.5, U8.11; no longer J10.1, J10.3, J11.1, J11.3, J11.4, J12.1, J12.3, J12.4, J15.3, J15.4, J15.5, J15.6, J18.4, J19.4, J20.6, J7.1, J7.3, J7.4, J8.1, J8.3, J8.4, J9.1, R35.2, U$22.GND, U$22.SYNC, U$3.GND, U$3.SYNC, U$5.GND, U$5.SYNC, U$8.19, U$8.20, U$8.25, U15.7, U16.4
- net IN1: now also H1.1.24
- net IN2: now also H1.1.23
- net IN3: now also H1.1.25
- net IN4: now also H1.1.26
- net IN5: now also H1.1.28
- net IN6: now also H1.1.27
- net IN7: now also H1.1.29
- net IN8: now also H1.1.30
- net LX: now also D3.C, R88.2
- net N$11: now also U21.1; no longer U$3.BST
- net N$12: now also U21.2; no longer U$3.SW
- net N$13: now also U$3.1, U$3.2, U$3.3, U$5.1, U$5.2, U$5.3; no longer U$6.1, U$6.2, U$6.3, U$7.1, U$7.2, U$7.3
- net N$15: now also U$5.4; no longer U$7.4
- net N$18: now also U$3.4; no longer U$6.4
- net N$25: now also U22.4; no longer U$5.RT
- net N$26: now also U$6.11; no longer U$8.11
- net N$27: now also U22.3; no longer U$5.INTVCC
- net N$28: now also U22.1; no longer U$5.BST
- net N$29: now also U22.2; no longer U$5.SW
- net N$30: now also U$6.8; no longer U$8.8
- net N$31: now also U23.4; no longer U$22.RT
- net N$32: now also U23.7; no longer U$22.TR/SS
- net N$33: now also U23.3; no longer U$22.INTVCC
- net N$34: now also U23.1; no longer U$22.BST
- net N$35: now also U23.2; no longer U$22.SW
- net N$36: now also U23.6; no longer U$22.FB
- net N$39: now also U$6.12; no longer U$8.12
- net N$43: now also U$6.21, U$6.22; no longer U$8.21, U$8.22
- net N$5: now also U$6.7; no longer U$8.7
- net N$51: now also U$6.17, U$6.18; no longer U$8.17, U$8.18
- net N$61: now also R66.1, R67.2, U16.4; no longer R57.2, U17.8
- net N$64: now also H1.P$4, R75.2; no longer R41.2
- net N$7: now also U21.3; no longer U$3.INTVCC
- net N$8: now also U21.4; no longer U$3.RT
- net N$9: now also U$6.2; no longer U$8.2
- net PCM_VBATT: now also R66.2; no longer C18.1, C22.1, C34.1, C40.1, R57.1, U$22.VIN, U$3.VIN, U$5.VIN, U17.1, U9.2, U9.3, U9.7
- net PG_5V_BURN: now also U23.8; no longer U$22.PG
- net RESET: now also H1.1.52, U19.5
- net SLEEP1: now also H1.1.42
- net SLEEP2: now also H1.1.48
- net SOLAR_IN1: no longer J7.2
- net SOLAR_IN2: no longer J8.2
- net SOLAR_IN3: no longer J9.2
- net SOLAR_IN4: no longer J10.2
- net SOLAR_IN5: no longer J11.2
- net SOLAR_IN6: no longer J12.2
- net SW: now also C96.1, R88.1
- net SW_12V_EN1: now also U8.10
- net SW_3V3_1: now also H1.2.19, J9.1
- net SW_3V3_2: now also H1.2.20
- net SW_5V_1: now also H1.2.13, J10.2
- net SW_5V_2: now also H1.2.15, J10.1
- net SW_5V_3: now also H1.2.16, J9.2
- net SW_5V_BURN_EN: now also U23.10; no longer U$22.EN/UV
- net SW_5V_EN4: no longer U8.4
- net TORQUE_1A: now also J7.1
- net TORQUE_1B: now also J7.2
- net TORQUE_2A: now also J7.4
- net TORQUE_2B: now also J7.3
- net TORQUE_3A: now also J8.1
- net TORQUE_3B: now also J8.2
- net TORQUE_4A: now also J8.4
- net TORQUE_4B: now also J8.3
- net TRQ1: now also H1.1.38
- net TRQ2: now also H1.1.44
- net USB_D+: now also U$6.24; no longer U$8.24
- net USB_D-: now also U$6.1; no longer U$8.1
- net USB_JUMP1: now also U$6.15, U$6.16; no longer U$8.15, U$8.16
- net USB_JUMP_BAT: now also U$6.13, U$6.14; no longer U$8.13, U$8.14
- net USB_VBUS: now also U$6.23; no longer U$8.23
- net VBATT: now also C18.1, C22.1, C34.1, C40.1, H1.2.35, H1.2.36, J16.1, R41.2, R57.2, R64.1, U17.1, U21.9, U22.9, U23.9, U9.2, U9.3, U9.7
- net VBURN1: now also U$3.5, U$3.6, U$3.7, U$3.8; no longer U$6.5, U$6.6, U$6.7, U$6.8
- net VBURN2: now also U$5.5, U$5.6, U$5.7, U$5.8; no longer U$7.5, U$7.6, U$7.7, U$7.8
- net VCC: no longer U$1.9
- net VIN3: no longer U8.6
- net VL: now also C89.2, C97.2, C98.2, CR1.1, CR2.1, CR3.1, CR4.1, CR5.1, CR6.1, CR7.1, R76.1, R87.2
- net VS: no longer C29.1, U15.5

Commit message: updated PDU v2 schematic
Parts:
- removed R41: 10k, HSFL_Main_Library:0805
- added J27, J28: 5037630491, Artemis:CON_5037630491
- added NT1, NT2, NT3: 0 H, HSFL_Main_Library:ELL4GG
- C65: value (none) -> 4.7 uF
- J21: value 5037630291 -> 5037630491; device Artemis:CON_5037630291 -> Artemis:CON_5037630491
- R18, R19, R20, R21: value 330 mΩ -> 330 m
- R39: value 55k -> 316k
- R40: value 100k -> 110k
- R65: value 190k -> 191k
- moved J21 167.7 mm to (-162.6, -29.2)
- moved R39 152.4 mm to (-167.6, 191.8)
- moved R69 147.3 mm to (-162.6, 196.8)
- moved R70 147.3 mm to (-167.6, 196.8)
- moved LED1 140.0 mm to (-19.1, 175.3)
- moved C20 139.7 mm to (-160.0, 175.3)
- moved C19 139.7 mm to (-154.9, 175.3)
- moved C21 139.7 mm to (-165.1, 175.3)
- moved C52 137.2 mm to (-152.4, 181.6)
- moved C53 137.2 mm to (-157.5, 181.6)
- moved C54 137.2 mm to (-162.6, 181.6)
- moved C55 137.2 mm to (-167.6, 181.6)
- moved C93 137.2 mm to (-152.4, 186.7)
- moved C94 137.2 mm to (-157.5, 186.7)
- moved C95 137.2 mm to (-162.6, 186.7)
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Connections:
- net BATTERY_DC renamed BATT_CHRG_DISP
- removed net BAT_CHARGE: J17.1
- removed net BC_OUT: C94.2, C95.2, H1.2.41, H1.2.42, H1.2.43, H1.2.44, U$1.3
- removed net KAPT_HEAT_IN: J26.1
- removed net N$101: U$1.22
- removed net N$19 (its old number): C27.1, C28.1, U2.13
- removed net N$20: C25.1, C26.1, U1.13
- removed net N$63: R39.2, R41.1
- removed net N$76: H1.1.49
- removed net N$77: H1.1.51
- removed net N$81: J18.4
- removed net N$82: J19.4
- removed net N$83: J20.6
- removed net PCM_VBATT: R66.2
- removed net SPI_MISO: J20.7, U14.48
- removed net SPI_MOSI: J20.3, U14.46
- removed net SPI_SCK: J20.5, U14.47
- removed net SPI_SD_CS: J20.1, R42.1, U14.49
- removed net SW_5V_EN4: U14.57
- removed net VCC: R35.1, U15.8
- removed net VS: R34.1, R36.1
- new net BATT_CHRG: C94.2, C95.2, H1.2.41, H1.2.42, H1.2.43, H1.2.44, J17.1, U$1.3
- new net MISO: J27.1, U14.48
- new net MOSI: J27.2, U14.46
- new net PB16: J28.1, U14.58
- new net PB17: J27.4, U14.59
- new net PB22: J28.3, U14.60
- new net PB23: J28.2, U14.61
- new net PDU_RX: H1.1.51, U14.83
- new net PDU_TX: H1.1.49, U14.82
- new net SCK: J27.3, U14.47
- new net SD_CS: J20.1, R42.1, U14.28
- new net SD_MISO: J20.7, U14.29
- new net SD_MOSI: J20.3, U14.26
- new net SD_SCK: J20.5, U14.27
- new net UART_TXD: H1.1.2
- net GND: now also C25.1, C26.1, C27.1, C28.1, J18.4, J19.4, J20.6, J21.5, J21.6, J27.5, J27.6, J28.4, J28.5, J28.6, J7.5, J7.6, J8.5, J8.6, NT1.P$1, NT2.P$1, NT3.P$1, U$1.22, U1.13, U2.13
- net GNDA: now also NT2.P$2, NT3.P$2
- net N$98: now also NT1.P$2
- net SOLAR_VS: now also R34.1, R36.1
- net SW_5V_3: now also J26.1
- net SW_VBATT_EN1: now also U14.57; no longer U14.58
- net UART2_RXD: now also H1.1.1
- net USB_D+: now also U14.85; no longer U14.86
- net USB_D-: now also U14.84; no longer U14.85
- net USB_VBUS: now also U14.32
- net VBATT: now also R35.1, R39.2, R66.2, R87.2, U15.8; no longer R41.2
- net VL: no longer R87.2
