File: hardware/Eagle Designs/PDU_v2/PDU_v2.1.sch (EAGLE design)
At the start: 245 parts, among them J1 5037630291, J10 5037630491, J11 UJ31-CH-G1-SMT-TR, J12 5037630291, J13 5037630291, J14 5037630291, J15 5037630291, J16 5037630291, J17 5037630291, J18 5037630491, J19 5037630291, J2 5037630291, J20 503182-1852, J22 5037630291, J23 5037630291, J24 5037630291, J25 5037630291, J27 5037630691, J3 5037630291, J4 5037630291, J5 5037630291, J6 5037630291, J7 5037630491, J8 5037630491, J9 5037630491, M1 BSZ100N06LS3, M2 BSZ100N06LS3, M3 BSZ033NE2LS5, M4 BSZ033NE2LS5, U1 DRV8847PWPR, U10 AO3404A, U11 IRLML2803PBFCT-ND, U12 IRLML2803PBFCT-ND, U13 LT8390EFE#PBF, U14 ATSAME51N19A-AF, U15 INA219BIDR, U16 MIC2514YM5-TR, U17 MAX16998AAUA+T, U18 TMP36FSZ, U2 DRV8847PWPR, U20 AO3404A, U21 LT8609A, U22 LT8609A, U23 BC848ALT1G, U24 AO3404A, U25 SI4835DDY-T1-GE3, U26 SI3493DDV-T1-GE3, U27 SI3493DDV-T1-GE3, U3 LTC1477CS8LINEAR_TECHNOLOGY_L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, U4 LTC1477CS8LINEAR_TECHNOLOGY_L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, U5 LTC1477CS8LINEAR_TECHNOLOGY_L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, U6 LTC1477CS8LINEAR_TECHNOLOGY_L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, U7 LTC1477CS8LINEAR_TECHNOLOGY_L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, U8 LT8609A, U9 LTC1477CS8LINEAR_TECHNOLOGY_L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, Y1 ABS07-32.768KHZ-T

Commit message: Completed OBC v4.1 (Finished); Updated PDU v2.1 (Unfinished)
Parts:
- added NT4: AIMC-0805-2N2S-T, PDUv2:AIMC-0805-2N2S-T
- R15: value 301 k -> 309 k
- R23: value 180 k -> 187 k
- R61: value 27 k -> 45.3 k
Connections:
- removed net RBF_OUT: J15.2, R83.1, U10.G
- new net PY_VBATT: J15.1, J16.1, R82.2, R83.1, U10.G, U24.D
- new net RBF_GND: NT4.2, R83.2, U10.S
- net GND: now also NT4.1; no longer R83.2, U10.S, U24.S
- net SW_12V_EN1: no longer U14.PC21
- net VBATT: now also J15.2, U24.S; no longer J15.1, J16.1, R82.2, U24.D
Other:
- note added: "BATT_CHRG is used for Battery Charging Circuit."
- note added: "CUS - Current Sensor"
- note added: "Functionality: Pin Removed = Open Circuit = PDU Powered On Pin In = Closed Circuit = PDU Powered Off"
- note added: "PY_VBATT is used for Pre-RBF Circuit."
- note added: "PY_VBATT: Power source directly from PyCubed Battery Board (Pre-RBF Circuit) VBATT: Power source that supplies to satellite (Post-RBF Circuit) J15 Connector: Solder these connections together"
- note added: "Temperature Sensor Analog Pins: AIN1 - PDU v2 AIN2 - Battery Board AIN3 - AIN 6 - Solar Panel"
- note added: "VBATT (Post-RBF Circuit) PY_VBATT (Pre-RBF Circuit)"
- note removed: "Pin Removed = Open Circuit = PDU v2 Powered On Pin In = Closed Circuit = PDU v2 Powered Off"

Commit message: updated OBC v4.1. with revision feedback
Other:
- note added: "12V Reg."
- note added: "12V Switch Regulator (PDU)"
- note added: "RPi (OBC)"
- note removed: "BBB"
Changed lines of the file:
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@@
 <text x="101.6" y="22.86" size="1.27" layer="97">VBATT (Post-RBF Circuit)
 PY_VBATT (Pre-RBF Circuit)</text>
+<text x="111.76" y="48.26" size="1.27" layer="94">Kapton Heater</text>
+<text x="114.3" y="50.8" size="1.27" layer="94">RPi (OBC)</text>
+<text x="114.3" y="38.1" size="1.27" layer="94">12V Reg.</text>
+<text x="190.5" y="48.26" size="1.27" layer="94">Breakout Power</text>
+<text x="109.22" y="43.18" size="1.27" layer="94">Breakout Power</text>
 </plain>
 <instances>
@@
 <pinref part="H1" gate="G$1" pin="2.25"/>
 <wire x1="142.24" y1="35.56" x2="134.62" y2="35.56" width="0.1524" layer="91"/>
-<label x="127" y="35.56" size="1.778" layer="95"/>
+<label x="124.46" y="35.56" size="1.778" layer="95"/>
 </segment>
 <segment>
@@
 <text x="182.88" y="20.32" size="5.08" layer="94">5V Switches</text>
 <text x="53.34" y="-30.48" size="2.54" layer="94">Breakout Power</text>
-<text x="170.18" y="-30.48" size="2.54" layer="94">BBB</text>
-<text x="160.02" y="-91.44" size="2.54" layer="94">Kapton Heater</text>
-<text x="246.38" y="-30.48" size="2.54" layer="94">Breakout Power</text>
+<text x="154.94" y="-30.48" size="2.54" layer="94">RPi (OBC)</text>
+<text x="154.94" y="-91.44" size="2.54" layer="94">Kapton Heater</text>
+<text x="238.76" y="-30.48" size="2.54" layer="94">Breakout Power</text>
 <text x="50.8" y="-106.68" size="1.778" layer="97">All cap are 0805 size.</text>
-<text x="246.38" y="-91.44" size="2.54" layer="94">12V Switch Regulator</text>
+<text x="233.68" y="-91.44" size="2.54" layer="94">12V Switch Regulator (PDU)</text>
 <text x="91.44" y="-119.38" size="5.08" layer="94">VBATT Switch</text>
 </plain>
