File: hardware/Eagle Designs/OBC_v4.21/OBCv4.21.sch (EAGLE design)
At the start: 36 parts, among them J1 MCX-J-P-H-RA-TH1, J10 5037630591, J11 5037630291, J12 5037630491, J13 5037630291, J14 5037630491, J2 5037630491, J3 5037630591, J4 5037630291, J5 5037630291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

Commit message: fixed OBC modular radio Radio Reset connection
Connections:
- removed net DIO0: U$1.8-TX2/IN1, U3.GPIO_0, U4.DIO0
- new net DIO1: U$1.8-TX2/IN1, U3.GPIO_1, U4.DIO1
- net RADIO_RESET: now also U3.GPIO_0; no longer U3.SDN
Other:
- note added: "Modular Radio DIO1 GPIO"
- note removed: "Modular Radio DIO0 GPIO"
Changed lines of the file:
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@@
 <text x="294.64" y="236.22" size="2.54" layer="91">Adafruit GPS Breakout
 (3.3V Power, UART5)</text>
-<text x="144.78" y="76.2" size="1.778" layer="94">Modular Radio DIO0 GPIO</text>
+<text x="144.78" y="76.2" size="1.778" layer="94">Modular Radio DIO1 GPIO</text>
 <text x="12.7" y="175.26" size="1.27" layer="97">I2C1 connected to
 PDU's Current Sensor I2C</text>
@@
 </segment>
 </net>
-<net name="DIO0" class="0">
+<net name="T_CS1" class="0">
+<segment>
+<pinref part="H1" gate="G$1" pin="2.4"/>
+<wire x1="200.66" y1="220.98" x2="208.28" y2="220.98" width="0.1524" layer="91"/>
+<label x="208.28" y="220.98" size="1.778" layer="95"/>
+</segment>
+<segment>
+<pinref part="U$1" gate="G$1" pin="9-OUT1C"/>
+<wire x1="121.92" y1="40.64" x2="124.46" y2="40.64" width="0.1524" layer="91"/>
+<label x="124.46" y="40.64" size="1.778" layer="95"/>
+</segment>
+</net>
+<net name="DIO1" class="0">
 <segment>
 <pinref part="U$1" gate="G$1" pin="8-TX2/IN1"/>
 <wire x1="121.92" y1="76.2" x2="124.46" y2="76.2" width="0.1524" layer="91"/>
 <label x="124.46" y="76.2" size="1.778" layer="95"/>
-</segment>
-</net>
-<net name="T_CS1" class="0">
-<segment>
-<pinref part="H1" gate="G$1" pin="2.4"/>
-<wire x1="200.66" y1="220.98" x2="208.28" y2="220.98" width="0.1524" layer="91"/>
-<label x="208.28" y="220.98" size="1.778" layer="95"/>
-</segment>
-<segment>
-<pinref part="U$1" gate="G$1" pin="9-OUT1C"/>
-<wire x1="121.92" y1="40.64" x2="124.46" y2="40.64" width="0.1524" layer="91"/>
-<label x="124.46" y="40.64" size="1.778" layer="95"/>
 </segment>
 </net>
@@
 <net name="RADIO_RESET" class="0">
 <segment>
-<pinref part="U3" gate="G$1" pin="SDN"/>
-<wire x1="167.64" y1="106.68" x2="162.56" y2="106.68" width="0.1524" layer="91"/>
-<label x="147.32" y="106.68" size="1.778" layer="95"/>
-</segment>
-<segment>
 <pinref part="U4" gate="G$1" pin="RESET"/>
 <wire x1="167.64" y1="53.34" x2="162.56" y2="53.34" width="0.1524" layer="91"/>
-<label x="144.78" y="53.34" size="1.778" layer="95"/>
+<label x="149.86" y="53.34" size="1.778" layer="95"/>
+</segment>
+<segment>
+<pinref part="U3" gate="G$1" pin="GPIO_0"/>
+<wire x1="205.74" y1="127" x2="210.82" y2="127" width="0.1524" layer="91"/>
+<label x="210.82" y="127" size="1.778" layer="95"/>
 </segment>
 </net>
@@
 </segment>
 </net>
-<net name="DIO0" class="0">
-<segment>
-<pinref part="U3" gate="G$1" pin="GPIO_0"/>
-<wire x1="205.74" y1="127" x2="210.82" y2="127" width="0.1524" layer="91"/>
-<label x="210.82" y="127" size="1.778" layer="95"/>
-</segment>
-<segment>
-<pinref part="U4" gate="G$1" pin="DIO0"/>
-<wire x1="205.74" y1="68.58" x2="210.82" y2="68.58" width="0.1524" layer="91"/>
-<label x="210.82" y="68.58" size="1.778" layer="95"/>
-</segment>
-</net>
 <net name="UART5_RXD" class="0">
 <segment>
@@
 </segment>
 </net>
+<net name="DIO1" class="0">
+<segment>
+<pinref part="U3" gate="G$1" pin="GPIO_1"/>
+<wire x1="205.74" y1="132.08" x2="210.82" y2="132.08" width="0.1524" layer="91"/>
+<label x="210.82" y="132.08" size="1.778" layer="95"/>
+</segment>
+<segment>
+<pinref part="U4" gate="G$1" pin="DIO1"/>
+<wire x1="205.74" y1="73.66" x2="210.82" y2="73.66" width="0.1524" layer="91"/>
+<label x="210.82" y="73.66" size="1.778" layer="95"/>
+</segment>
+</net>

Commit message: uploaded official OBC v4.21
Parts:
- added R3: 0, HSFL_Main_Library:RESISTOR0805-RES
Connections:
- new net N$9: R3.1, U3.GPIO_0
- net RADIO_RESET: now also R3.2; no longer U3.GPIO_0
Changed lines of the file:
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@@
 <part name="U3" library="RFM RADIOS" deviceset="RFM23BP" device=""/>
 <part name="U4" library="RFM RADIOS" deviceset="RFM69HCW" device=""/>
+<part name="R3" library="HSFL_Main_Library" deviceset="RESISTOR" device="0805-RES" value="0"/>
 </parts>
 <sheets>
@@
 <attribute name="VALUE" x="172.72" y="38.608" size="1.778" layer="96"/>
 </instance>
+<instance part="R3" gate="G$1" x="218.44" y="127" smashed="yes">
+<attribute name="NAME" x="214.63" y="128.4986" size="1.778" layer="95"/>
+<attribute name="VALUE" x="222.25" y="130.302" size="1.778" layer="96" rot="R180"/>
+</instance>
 </instances>
 <busses>
@@
 </segment>
 <segment>
-<pinref part="U3" gate="G$1" pin="GPIO_0"/>
-<wire x1="205.74" y1="127" x2="210.82" y2="127" width="0.1524" layer="91"/>
-<label x="210.82" y="127" size="1.778" layer="95"/>
+<pinref part="R3" gate="G$1" pin="2"/>
+<wire x1="223.52" y1="127" x2="226.06" y2="127" width="0.1524" layer="91"/>
+<label x="226.06" y="127" size="1.778" layer="95"/>
 </segment>
 </net>
@@
 </segment>
 </net>
+<net name="N$9" class="0">
+<segment>
+<pinref part="U3" gate="G$1" pin="GPIO_0"/>
+<pinref part="R3" gate="G$1" pin="1"/>
+<wire x1="205.74" y1="127" x2="213.36" y2="127" width="0.1524" layer="91"/>
+</segment>
+</net>
