File: hardware/Eagle Designs/PDU/PDUv2.2/PDU_v2.2.sch (EAGLE design)
At the start: 274 parts, among them J1 5037630291, J10 5037630491, J11 UJ31-CH-G1-SMT-TR, J12 5037630291, J13 5037630291, J14 5037630291, J15 5037630291, J16 5037630291, J17 5037630291, J18 5037630491, J19 5037630291, J2 5037630291, J20 503182-1852, J22 5037630291, J23 5037630291, J24 5037630291, J25 5037630291, J27 5037630691, J28 68016-202HLF, J3 5037630291, J4 5037630291, J5 5037630291, J6 5037630291, J7 5037630491, J8 5037630491, J9 5037630491, M1 BSZ100N06LS3, M2 BSZ100N06LS3, M3 BSZ033NE2LS5, M4 BSZ033NE2LS5, U1 DRV8847PWPR, U10 AO3404A, U11 IRLML2803PBFCT-ND, U12 IRLML2803PBFCT-ND, U13 LT8390EFE#PBF, U14 ATSAME51N19A-AF, U15 INA219BIDR, U16 MIC2514YM5-TR, U17 MAX16998AAUA+T, U18 TMP36FSZ, U2 DRV8847PWPR, U20 LTC4012IUFPBF, U21 LT8609A, U22 LT8609A, U23 BC848ALT1G, U24 AO3404A, U25 SI4835DDY-T1-GE3, U26 SI3493DDV-T1-GE3, U27 SI3493DDV-T1-GE3, U28 SI4431BDY-T1-E3, U29 AO4818B, U3 LTC1477CS8LINEAR_TECHNOLOGY_L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, U30 INA219BIDR, U31 INA219BIDR, U32 INA219BIDR, U33 INA219BIDR, U35 LND01K1-G, U4 LTC1477CS8LINEAR_TECHNOLOGY_L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, U5 LTC1477CS8LINEAR_TECHNOLOGY_L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, U6 LTC1477CS8LINEAR_TECHNOLOGY_L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, U7 LTC1477CS8LINEAR_TECHNOLOGY_L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, U8 LT8609A, U9 LTC1477CS8LINEAR_TECHNOLOGY_L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, Y1 ABS07-32.768KHZ-T

Commit message: updated PDU v2.2
Parts:
- removed NT1: AIMC-0805-2N2S-T, PDUv2:AIMC-0805-2N2S-T
- removed R82, R83: 1 M, HSFL_Main_Library:RESISTOR0805-RES
- removed R93: 10 k, HSFL_Main_Library:RESISTOR0805-RES
- removed U10, U24: AO3404A, Artemis:AO3404A
- removed U35: LND01K1-G, PDU:LND01K1-G
Connections:
- removed net N$20: R82.1, U10.D, U24.G
- removed net N$60: R93.1, U35.DRAIN
- removed net RBF_GND: NT1.2, R83.2, U10.S
- removed net RBF_SW: J15.2, R83.1, U10.G
- removed net SOLAR_IN5_LOAD: D10.12
- removed net SOLAR_IN6_LOAD: D11.12
- net BUS_3V3: now also C64.1, D2.VDD
- net BUS_5V: no longer C64.1, D2.VDD
- net CS_VBATT: now also J15.2; no longer U24.S
- net GND: no longer NT1.1, R93.2
- net PY_VBATT: no longer R82.2, U24.D
- net SOLAR_IN5: now also D10.12
- net SOLAR_IN6: now also D11.12
- net SW_5V_1: no longer U35.SOURCE
- net SW_5V_EN1: no longer U35.GATE
Other:
- note added: "Insert Before Flight"
- note added: "PY_VBATT: Power source directly from PyCubed Battery Board CS_VBATT: Power source goes directly to current sensor for readings"
- note removed: "Depletion MOSFETs"
- note removed: "Functionality: Pin Removed = Open Circuit = PDU Powered On Pin In = Closed Circuit = PDU Powered Off"
- note removed: "Male Connector (MC) External Part Not Shown MC in (Pin In) MC disconnected (Pin Out)"
- note removed: "PY_VBATT: Power source directly from PyCubed Battery Board (Pre-RBF Circuit) CS_VBATT: Power source goes directly to current sensor for readings (Post-RBF Circuit)"
- note removed: "Remove Before Flight (RBF) Circuit"
- moved on the sheet: J15
