File: hardware/Eagle Designs/PDU/PDUv2.2/PDU_v2.2.brd (EAGLE design)
At the start: 90.2 x 95.5 mm, 267 parts, among them J1 5037630291, J10 5037630491, J11 UJ31-CH-G1-SMT-TR, J12 5037630291, J13 5037630291, J14 5037630291, J15 5037630291, J16 5037630291, J17 5037630291, J18 5037630491, J19 5037630291, J2 5037630291, J20 503182-1852, J22 5037630291, J23 5037630291, J24 5037630291, J25 5037630291, J27 5037630691, J28 68016-202HLF, J3 5037630291, J4 5037630291, J5 5037630291, J6 5037630291, J7 5037630491, J8 5037630491, J9 5037630491, M1 BSZ100N06LS3, M2 BSZ100N06LS3, M3 BSZ033NE2LS5, M4 BSZ033NE2LS5, U1 DRV8847PWPR, U11 IRLML2803PBFCT-ND, U12 IRLML2803PBFCT-ND, U13 LT8390EFE#PBF, U14 ATSAME51N19A-AF, U15 INA219BIDR, U16 MIC2514YM5-TR, U17 MAX16998AAUA+T, U18 TMP36FSZ, U2 DRV8847PWPR, U20 LTC4012IUFPBF, U21 LT8609A, U22 LT8609A, U23 BC848ALT1G, U25 SI4835DDY-T1-GE3, U26 SI3493DDV-T1-GE3, U27 SI3493DDV-T1-GE3, U28 SI4431BDY-T1-E3, U29 AO4818B, U3 LTC1477CS8LINEAR_TECHNOLOGY_L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, U30 INA219BIDR, U31 INA219BIDR, U32 INA219BIDR, U33 INA219BIDR, U4 LTC1477CS8LINEAR_TECHNOLOGY_L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, U5 LTC1477CS8LINEAR_TECHNOLOGY_L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, U6 LTC1477CS8LINEAR_TECHNOLOGY_L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, U7 LTC1477CS8LINEAR_TECHNOLOGY_L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, U8 LT8609A, U9 LTC1477CS8LINEAR_TECHNOLOGY_L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, Y1 ABS07-32.768KHZ-T

Commit message: fixed PDU for manufacturing
Routing:
- net INH_SW1_COM: track 290.9 -> 290.2 mm
Changed lines of the file:
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@@
 <setting verticaltext="up"/>
 </settings>
-<grid distance="0.5" unitdist="mm" unit="mm" style="lines" multiple="1" display="yes" altdistance="0.5" altunitdist="mil" altunit="mm"/>
+<grid distance="0.01" unitdist="mil" unit="mil" style="lines" multiple="1" display="yes" altdistance="0.01" altunitdist="mil" altunit="mil"/>
 <layers>
 <layer number="1" name="Top" color="4" fill="1" visible="yes" active="yes"/>
@@
 <wire x1="12.743" y1="7.663" x2="11.43" y2="6.35" width="0.762" layer="1"/>
 <via x="83.7184" y="13.97" extent="1-16" drill="0.3556"/>
-<wire x1="11.43" y1="6.35" x2="12.6402" y2="5.1398" width="0.762" layer="2"/>
-<wire x1="12.6402" y1="5.1398" x2="78.1298" y2="5.1398" width="0.5" layer="2"/>
-<wire x1="83.7184" y1="10.7284" x2="78.1298" y2="5.1398" width="0.762" layer="2"/>
-<wire x1="83.7184" y1="10.7284" x2="83.7184" y2="13.97" width="0.762" layer="2"/>
+<wire x1="11.43" y1="6.35" x2="11.576703125" y2="6.203296875" width="0.762" layer="2"/>
+<wire x1="11.576703125" y1="6.203296875" x2="79.6571" y2="6.203296875" width="0.5" layer="2"/>
+<wire x1="83.7184" y1="10.264596875" x2="79.6571" y2="6.203296875" width="0.5" layer="2"/>
+<wire x1="83.7184" y1="10.264596875" x2="83.7184" y2="13.97" width="0.762" layer="2"/>
 <wire x1="84.7598" y1="81.7308" x2="84.64" y2="81.611" width="0.762" layer="1"/>
 <wire x1="84.7598" y1="81.7308" x2="84.7598" y2="82.6008" width="0.762" layer="1"/>
