File: hardware/Eagle Designs/OBC_v4.23/OBCv4.23.brd (EAGLE design)
At the start: 90.2 x 95.5 mm, 38 parts, among them J1 MCX-J-P-H-RA-TH1, J10 5037630591, J11 5037630291, J12 5037630491, J13 5037630291, J14 5037630491, J2 5037630491, J3 5037630591, J4 5037630291, J5 5037630291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

Commit message: updated and finalized OBC V4.23
Parts:
- removed R7: 0, HSFL_Main_Library:1206
- added R9: 0, HSFL_Main_Library:R2512
- R8: device HSFL_Main_Library:1206 -> HSFL_Main_Library:R2512
- moved R8 6.66 mm to (40.8, 40.3)
Connections:
- net +3V3_VCC: now also R9.2; no longer R8.2
- net 5V_BUS: now also R8.2; no longer R7.2
- net N$10: now also R9.1; no longer R8.1
- net N$9: now also R8.1; no longer R7.1
Routing:
- net 5V_BUS: track 138.0 -> 134.5 mm
- net +3V3_VCC: track 332.5 -> 329.7 mm
- net N$10: track 27.4 -> 29.0 mm
- net N$9: track 32.3 -> 31.2 mm
