File: hardware/Eagle Designs/OBC_v4.23/OBCv4.23.sch (EAGLE design)
At the start: 38 parts, among them J1 MCX-J-P-H-RA-TH1, J10 5037630591, J11 5037630291, J12 5037630491, J13 5037630291, J14 5037630491, J2 5037630491, J3 5037630591, J4 5037630291, J5 5037630291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

Commit message: updated and finalized OBC V4.23
Parts:
- removed R7: 0, HSFL_Main_Library:RESISTOR1206
- added R9: 0, HSFL_Main_Library:RESISTOR2512
- R8: device HSFL_Main_Library:RESISTOR1206 -> HSFL_Main_Library:RESISTOR2512
Connections:
- net +3V3_VCC: now also R9.2; no longer R8.2
- net 5V_BUS: now also R8.2; no longer R7.2
- net N$10: now also R9.1; no longer R8.1
- net N$9: now also R8.1; no longer R7.1
Other:
- moved on the sheet: R8
Changed lines of the file:
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@@
 <part name="U3" library="RFM RADIOS" deviceset="RFM23BP" device=""/>
 <part name="U4" library="RFM RADIOS" deviceset="RFM69HCW" device=""/>
-<part name="R8" library="HSFL_Main_Library" deviceset="RESISTOR" device="1206" value="0"/>
-<part name="R7" library="HSFL_Main_Library" deviceset="RESISTOR" device="1206" value="0"/>
+<part name="R8" library="HSFL_Main_Library" deviceset="RESISTOR" device="2512" value="0"/>
+<part name="R9" library="HSFL_Main_Library" deviceset="RESISTOR" device="2512" value="0"/>
 </parts>
 <sheets>
@@
 <attribute name="VALUE" x="172.72" y="38.608" size="1.778" layer="96"/>
 </instance>
-<instance part="R8" gate="G$1" x="215.9" y="63.5" smashed="yes">
+<instance part="R8" gate="G$1" x="215.9" y="121.92" smashed="yes">
+<attribute name="NAME" x="212.09" y="123.4186" size="1.778" layer="95"/>
+<attribute name="VALUE" x="217.17" y="123.698" size="1.778" layer="96"/>
+</instance>
+<instance part="R9" gate="G$1" x="215.9" y="63.5" smashed="yes">
 <attribute name="NAME" x="212.09" y="64.9986" size="1.778" layer="95"/>
-<attribute name="VALUE" x="212.09" y="60.198" size="1.778" layer="96"/>
-</instance>
-<instance part="R7" gate="G$1" x="215.9" y="121.92" smashed="yes">
-<attribute name="NAME" x="212.09" y="123.4186" size="1.778" layer="95"/>
-<attribute name="VALUE" x="212.09" y="118.618" size="1.778" layer="96"/>
+<attribute name="VALUE" x="219.71" y="65.278" size="1.778" layer="96"/>
 </instance>
 </instances>
@@
 </segment>
 <segment>
-<wire x1="220.98" y1="63.5" x2="226.06" y2="63.5" width="0.1524" layer="91"/>
-<label x="226.06" y="63.5" size="1.778" layer="95"/>
-<pinref part="R8" gate="G$1" pin="2"/>
+<pinref part="R9" gate="G$1" pin="2"/>
+<wire x1="220.98" y1="63.5" x2="223.52" y2="63.5" width="0.1524" layer="91"/>
+<label x="220.98" y="63.5" size="1.778" layer="95"/>
 </segment>
 </net>
@@
 <net name="5V_BUS" class="0">
 <segment>
-<wire x1="220.98" y1="121.92" x2="228.6" y2="121.92" width="0.1524" layer="91"/>
-<label x="228.6" y="121.92" size="1.778" layer="95"/>
-<pinref part="R7" gate="G$1" pin="2"/>
+<pinref part="R8" gate="G$1" pin="2"/>
+<wire x1="220.98" y1="121.92" x2="226.06" y2="121.92" width="0.1524" layer="91"/>
+<label x="226.06" y="121.92" size="1.778" layer="95"/>
 </segment>
 </net>
@@
 <net name="N$9" class="0">
 <segment>
+<pinref part="R8" gate="G$1" pin="1"/>
+<wire x1="210.82" y1="121.92" x2="205.74" y2="121.92" width="0.1524" layer="91"/>
 <pinref part="U3" gate="G$1" pin="VCC"/>
-<pinref part="R7" gate="G$1" pin="1"/>
-<wire x1="205.74" y1="121.92" x2="210.82" y2="121.92" width="0.1524" layer="91"/>
 </segment>
 </net>
 <net name="N$10" class="0">
 <segment>
-<pinref part="R8" gate="G$1" pin="1"/>
+<pinref part="R9" gate="G$1" pin="1"/>
 <pinref part="U4" gate="G$1" pin="3V3"/>
 <wire x1="210.82" y1="63.5" x2="205.74" y2="63.5" width="0.1524" layer="91"/>
