File: hardware/Eagle Designs/OBC/OBC_V4.24_w:_RFplane/OBCv4.24.brd (EAGLE design)
At the start: 90.2 x 95.5 mm, 38 parts, among them J1 MCX-J-P-H-RA-TH1, J10 5037630591, J11 5037630291, J12 5037630491, J13 5037630291, J14 5037630491, J2 5037630491, J3 5037630591, J4 5037630291, J5 5037630291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

Commit message: cleaned up a wire stub on OBC 4.24 and copied OBC for RF with ground plane
Routing:
- net UART6_TX: track 0.00 -> 59.0 mm, vias 0 -> 1
- net RADIO_RESET: track 84.7 -> 130.7 mm
- net NIRQ: track 53.4 -> 90.8 mm
- net UART6_RX: track 29.6 -> 60.3 mm, vias 0 -> 1
- net ANT_CONN: track 114.6 -> 108.1 mm
Changed lines of the file:
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@@
 <wire x1="41.76" y1="25.88" x2="37.87" y2="21.99" width="0.6" layer="2"/>
 <wire x1="37.87" y1="21.99" x2="32.07" y2="21.99" width="0.6" layer="2"/>
-<wire x1="41.1" y1="56.46" x2="36.36" y2="61.2" width="0.4" layer="16"/>
-<wire x1="41.1" y1="56.46" x2="41.1" y2="46.01" width="0.4" layer="16"/>
 <contactref element="U3" pad="14"/>
 <wire x1="32.67" y1="19.1" x2="35.65" y2="19.1" width="0.5" layer="16"/>
@@
 <wire x1="35.65" y1="19.1" x2="41.44908125" y2="19.1" width="0.5" layer="16"/>
 <wire x1="41.44908125" y1="19.1" x2="41.76" y2="19.41091875" width="0.5" layer="16"/>
-<wire x1="48.32" y1="38.79" x2="48.32" y2="35.57" width="0.4" layer="16"/>
-<wire x1="41.1" y1="46.01" x2="48.32" y2="38.79" width="0.4" layer="16"/>
-<wire x1="41.76" y1="25.88" x2="42.97" y2="25.88" width="0.4" layer="16"/>
-<wire x1="42.97" y1="25.88" x2="44.82" y2="27.73" width="0.4" layer="16"/>
-<wire x1="44.82" y1="27.73" x2="46.17" y2="27.73" width="0.4" layer="16"/>
-<wire x1="48.38" y1="29.94" x2="46.17" y2="27.73" width="0.4" layer="16"/>
-<wire x1="48.3" y1="35.59" x2="48.32" y2="35.57" width="0.3" layer="16"/>
-<wire x1="48.32" y1="35.57" x2="48.38" y2="35.51" width="0.3" layer="16"/>
-<wire x1="48.38" y1="35.51" x2="48.38" y2="29.94" width="0.3" layer="16"/>
 <contactref element="U$1" pad="32-OUT1B"/>
-<wire x1="36.36" y1="61.2" x2="74.46" y2="64.11" width="0" layer="19" extent="16-16"/>
+<wire x1="41.76" y1="25.88" x2="44.87" y2="22.77" width="0.508" layer="1"/>
+<wire x1="44.87" y1="22.77" x2="67.97" y2="22.77" width="0.508" layer="1"/>
+<wire x1="67.97" y1="22.77" x2="81.31" y2="36.11" width="0.508" layer="1"/>
+<wire x1="81.31" y1="36.11" x2="84.74" y2="36.11" width="0.508" layer="1"/>
+<wire x1="84.74" y1="36.11" x2="86.96" y2="38.33" width="0.508" layer="1"/>
+<wire x1="86.96" y1="38.33" x2="86.96" y2="63" width="0.508" layer="1"/>
+<wire x1="86.96" y1="63" x2="85.81" y2="64.15" width="0.508" layer="1"/>
+<wire x1="85.81" y1="64.15" x2="74.5" y2="64.15" width="0.508" layer="1"/>
+<wire x1="74.5" y1="64.15" x2="74.46" y2="64.11" width="0.508" layer="1"/>
 </signal>
 <signal name="3V3_BUS">
@@
 <wire x1="78.27" y1="5.32" x2="34.64" y2="5.32" width="0.8" layer="15"/>
 <wire x1="31.36" y1="8.6" x2="34.64" y2="5.32" width="0.8" layer="15"/>
-<wire x1="35.65" y1="9.1" x2="38.805" y2="9.1" width="0.5" layer="16"/>
-<wire x1="35.4" y1="9.14" x2="38.805" y2="9.1" width="0.5" layer="16"/>
+<wire x1="35.65" y1="9.1" x2="35.4" y2="9.14" width="0" layer="19" extent="16-16"/>
 </signal>
 <signal name="N$16">
@@
 <wire x1="77.86" y1="13.87" x2="79.48" y2="15.49" width="0.7" layer="15"/>
 <wire x1="79.48" y1="15.49" x2="79.48" y2="34.63" width="0.7" layer="15"/>
-<via x="64.66" y="40.53" extent="1-16" drill="0.35"/>
-<wire x1="64.66" y1="40.53" x2="64.6" y2="40.47" width="0.7" layer="2"/>
-<wire x1="64.6" y1="40.47" x2="62.54" y2="40.47" width="0.7" layer="2"/>
-<wire x1="73.58" y1="40.53" x2="64.66" y2="40.53" width="0.7" layer="15"/>
 <wire x1="79.48" y1="34.63" x2="73.58" y2="40.53" width="0.7" layer="15"/>
 <contactref element="U$1" pad="40-A16/CS1"/>
-<wire x1="62.54" y1="40.47" x2="56.68" y2="79.35" width="0" layer="19" extent="1-2"/>
+<wire x1="73.58" y1="40.53" x2="73.25" y2="40.86" width="0.8128" layer="15"/>
+<wire x1="73.25" y1="62.76" x2="73.25" y2="40.86" width="0.8128" layer="15"/>
+<wire x1="61.2583" y1="73.0588" x2="56.68" y2="77.6371" width="0.6096" layer="1"/>
+<wire x1="56.68" y1="77.6371" x2="56.68" y2="79.35" width="0.6096" layer="1"/>
+<wire x1="61.2583" y1="73.0588" x2="62.9712" y2="73.0588" width="0.6096" layer="1"/>
+<via x="65.84" y="73.05" extent="1-16" drill="0.35"/>
+<wire x1="62.9712" y1="73.0588" x2="65.8312" y2="73.0588" width="0.508" layer="1"/>
+<wire x1="65.8312" y1="73.0588" x2="65.84" y2="73.05" width="0.508" layer="1"/>
+<wire x1="65.84" y1="73.05" x2="73.2488" y2="65.6412" width="0.508" layer="15"/>
+<wire x1="73.2488" y1="62.7612" x2="73.25" y2="62.76" width="0.508" layer="15"/>
+<wire x1="73.2488" y1="65.6412" x2="73.2488" y2="62.7612" width="0.508" layer="15"/>
 </signal>
 <signal name="RX_ON">
@@
 <wire x1="26.78" y1="37.33" x2="27.9" y2="38.45" width="0.5" layer="1"/>
 <wire x1="27.9" y1="38.45" x2="34.35" y2="38.45" width="0.5" layer="1"/>
-<wire x1="34.35" y1="38.45" x2="48.56" y2="52.66" width="0.5" layer="1"/>
-<wire x1="48.56" y1="52.66" x2="36.36" y2="64.11" width="0" layer="19" extent="1-1"/>
+<wire x1="45.0646" y1="53.1560375" x2="45.24" y2="53.3314375" width="0.6096" layer="1"/>
+<wire x1="34.35" y1="38.45" x2="45.0646" y2="49.1646" width="0.6096" layer="1"/>
+<wire x1="45.0646" y1="49.1646" x2="45.0646" y2="53.1560375" width="0.6096" layer="1"/>
+<via x="44.37" y="72.58" extent="1-16" drill="0.35"/>
+<wire x1="45.24" y1="71.71" x2="44.37" y2="72.58" width="0.6096" layer="1"/>
+<wire x1="45.24" y1="53.3314375" x2="45.24" y2="71.71" width="0.6096" layer="1"/>
+<wire x1="44.37" y1="72.58" x2="44.37" y2="72.12" width="0.6096" layer="15"/>
+<wire x1="44.37" y1="72.12" x2="36.36" y2="64.11" width="0.6096" layer="15"/>
 </signal>
 <signal name="UART6_TX">
 <contactref element="U$1" pad="8-TX2/IN1"/>
 <contactref element="X1" pad="10"/>
-<wire x1="29.32" y1="35.814" x2="38.9" y2="64.11" width="0" layer="19" extent="1-1"/>
+<wire x1="50.24" y1="67.8" x2="50.24" y2="67.92" width="0.508" layer="1"/>
+<via x="47.19" y="70.57" extent="1-16" drill="0.35"/>
+<wire x1="50.24" y1="67.8" x2="47.47" y2="70.57" width="0.508" layer="1"/>
+<wire x1="47.47" y1="70.57" x2="47.19" y2="70.57" width="0.508" layer="1"/>
+<wire x1="47.19" y1="70.57" x2="43.02" y2="66.4" width="0.508" layer="15"/>
+<wire x1="41.19" y1="66.4" x2="38.9" y2="64.11" width="0.508" layer="15"/>
+<wire x1="43.02" y1="66.4" x2="41.19" y2="66.4" width="0.508" layer="15"/>
+<wire x1="50.24" y1="51.63" x2="36.31" y2="37.7" width="0.508" layer="1"/>
+<wire x1="36.2712" y1="37.7388" x2="36.31" y2="37.7" width="0.508" layer="1"/>
+<wire x1="50.24" y1="67.8" x2="50.24" y2="51.63" width="0.508" layer="1"/>
+<wire x1="36.31" y1="37.7" x2="35.86" y2="37.25" width="0.508" layer="1"/>
+<wire x1="30.756" y1="37.25" x2="29.32" y2="35.814" width="0.508" layer="1"/>
+<wire x1="35.86" y1="37.25" x2="30.756" y2="37.25" width="0.508" layer="1"/>
 </signal>
 </signals>
