File: hardware/Eagle Designs/OBC/OBC_V4.24_RFplane/OBCv4.24.sch (EAGLE design)
At the start: 38 parts, among them J1 MCX-J-P-H-RA-TH1, J10 5037630591, J11 5037630291, J12 5037630491, J13 5037630291, J14 5037630491, J2 5037630491, J3 5037630591, J4 5037630291, J5 5037630291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

Commit message: Added RF plane to OBCv4.24
Parts:
- added R3: 1M, HSFL_Main_Library:RESISTOR0805-RES
Connections:
- new net GPS_GND: R6.1, U6.GND_RF, U6.P$22, U6.P$24, U6.P$25, U6.P$27, U6.P$28, U6.P$29, U6.P$31, U6.P$33
- net GND: now also R3.2; no longer J1.2, U3.GND1, U3.GND2, U3.GND3, U4.GND1, U4.GND2, U4.GND3
- net RF_GND: now also J1.2, R3.1, U3.GND1, U3.GND2, U3.GND3, U4.GND1, U4.GND2, U4.GND3; no longer R6.1, U6.GND_RF, U6.P$22, U6.P$24, U6.P$25, U6.P$27, U6.P$28, U6.P$29, U6.P$31, U6.P$33
Changed lines of the file:
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@@
 <part name="R8" library="HSFL_Main_Library" deviceset="RESISTOR" device="2512" value="0"/>
 <part name="R9" library="HSFL_Main_Library" deviceset="RESISTOR" device="2512" value="0"/>
+<part name="R3" library="HSFL_Main_Library" deviceset="RESISTOR" device="0805-RES" value="1M"/>
 </parts>
 <sheets>
@@
 <attribute name="VALUE" x="219.71" y="65.278" size="1.778" layer="96"/>
 </instance>
+<instance part="R3" gate="G$1" x="205.74" y="30.48" smashed="yes">
+<attribute name="NAME" x="201.93" y="31.9786" size="1.778" layer="95"/>
+<attribute name="VALUE" x="201.93" y="27.178" size="1.778" layer="96"/>
+</instance>
 </instances>
 <busses>
@@
 </segment>
 <segment>
-<pinref part="J1" gate="G$1" pin="2"/>
-<wire x1="233.68" y1="45.72" x2="228.6" y2="45.72" width="0.1524" layer="91"/>
-<label x="223.52" y="45.72" size="1.778" layer="95"/>
-</segment>
-<segment>
-<pinref part="U3" gate="G$1" pin="GND1"/>
-<wire x1="167.64" y1="137.16" x2="162.56" y2="137.16" width="0.1524" layer="91"/>
-<label x="157.48" y="137.16" size="1.778" layer="95"/>
-</segment>
-<segment>
-<pinref part="U3" gate="G$1" pin="GND2"/>
-<wire x1="167.64" y1="101.6" x2="162.56" y2="101.6" width="0.1524" layer="91"/>
-<label x="157.48" y="101.6" size="1.778" layer="95"/>
-</segment>
-<segment>
-<pinref part="U3" gate="G$1" pin="GND3"/>
-<wire x1="205.74" y1="106.68" x2="210.82" y2="106.68" width="0.1524" layer="91"/>
-<label x="210.82" y="106.68" size="1.778" layer="95"/>
-</segment>
-<segment>
-<pinref part="U4" gate="G$1" pin="GND1"/>
-<wire x1="167.64" y1="78.74" x2="162.56" y2="78.74" width="0.1524" layer="91"/>
-<label x="157.48" y="78.74" size="1.778" layer="95"/>
-</segment>
-<segment>
-<pinref part="U4" gate="G$1" pin="GND2"/>
-<wire x1="167.64" y1="43.18" x2="162.56" y2="43.18" width="0.1524" layer="91"/>
-<label x="157.48" y="43.18" size="1.778" layer="95"/>
-</segment>
-<segment>
-<pinref part="U4" gate="G$1" pin="GND3"/>
-<wire x1="205.74" y1="48.26" x2="210.82" y2="48.26" width="0.1524" layer="91"/>
-<label x="210.82" y="48.26" size="1.778" layer="95"/>
+<pinref part="R3" gate="G$1" pin="2"/>
+<wire x1="210.82" y1="30.48" x2="213.36" y2="30.48" width="0.1524" layer="91"/>
+<label x="213.36" y="30.48" size="1.778" layer="95"/>
 </segment>
 </net>
@@
 <net name="RF_GND" class="0">
 <segment>
+<pinref part="J1" gate="G$1" pin="2"/>
+<wire x1="233.68" y1="45.72" x2="228.6" y2="45.72" width="0.1524" layer="91"/>
+<label x="228.6" y="45.72" size="1.778" layer="95" rot="MR0"/>
+</segment>
+<segment>
+<pinref part="U3" gate="G$1" pin="GND1"/>
+<wire x1="167.64" y1="137.16" x2="162.56" y2="137.16" width="0.1524" layer="91"/>
+<label x="157.48" y="137.16" size="1.778" layer="95"/>
+</segment>
+<segment>
+<pinref part="U3" gate="G$1" pin="GND2"/>
+<wire x1="167.64" y1="101.6" x2="162.56" y2="101.6" width="0.1524" layer="91"/>
+<label x="157.48" y="101.6" size="1.778" layer="95"/>
+</segment>
+<segment>
+<pinref part="U3" gate="G$1" pin="GND3"/>
+<wire x1="205.74" y1="106.68" x2="210.82" y2="106.68" width="0.1524" layer="91"/>
+<label x="210.82" y="106.68" size="1.778" layer="95"/>
+</segment>
+<segment>
+<pinref part="U4" gate="G$1" pin="GND1"/>
+<wire x1="167.64" y1="78.74" x2="162.56" y2="78.74" width="0.1524" layer="91"/>
+<label x="157.48" y="78.74" size="1.778" layer="95"/>
+</segment>
+<segment>
+<pinref part="U4" gate="G$1" pin="GND2"/>
+<wire x1="167.64" y1="43.18" x2="162.56" y2="43.18" width="0.1524" layer="91"/>
+<label x="157.48" y="43.18" size="1.778" layer="95"/>
+</segment>
+<segment>
+<pinref part="U4" gate="G$1" pin="GND3"/>
+<wire x1="205.74" y1="48.26" x2="210.82" y2="48.26" width="0.1524" layer="91"/>
+<label x="210.82" y="48.26" size="1.778" layer="95"/>
+</segment>
+<segment>
+<pinref part="R3" gate="G$1" pin="1"/>
+<wire x1="200.66" y1="30.48" x2="198.12" y2="30.48" width="0.1524" layer="91"/>
+<label x="198.12" y="30.48" size="1.778" layer="95" rot="MR0"/>
+</segment>
+</net>
+<net name="UART5_RXD" class="0">
+<segment>
+<pinref part="U6" gate="G$1" pin="GPS_RXDO"/>
+<wire x1="109.22" y1="121.92" x2="121.92" y2="121.92" width="0.1524" layer="91"/>
+<label x="114.3" y="121.92" size="1.778" layer="95"/>
+</segment>
+</net>
+<net name="DIO1" class="0">
+<segment>
+<pinref part="U3" gate="G$1" pin="GPIO_1"/>
+<wire x1="205.74" y1="132.08" x2="210.82" y2="132.08" width="0.1524" layer="91"/>
+<label x="210.82" y="132.08" size="1.778" layer="95"/>
+</segment>
+<segment>
+<pinref part="U4" gate="G$1" pin="DIO1"/>
+<wire x1="205.74" y1="73.66" x2="210.82" y2="73.66" width="0.1524" layer="91"/>
+<label x="210.82" y="73.66" size="1.778" layer="95"/>
+</segment>
+</net>
+<net name="NIRQ" class="0">
+<segment>
+<pinref part="U3" gate="G$1" pin="NIRQ"/>
+<wire x1="167.64" y1="111.76" x2="162.56" y2="111.76" width="0.1524" layer="91"/>
+<label x="157.48" y="111.76" size="1.778" layer="95"/>
+</segment>
+</net>
+<net name="RX_ON" class="0">
+<segment>
+<pinref part="U3" gate="G$1" pin="RXON"/>
+<wire x1="205.74" y1="116.84" x2="210.82" y2="116.84" width="0.1524" layer="91"/>
+<label x="210.82" y="116.84" size="1.778" layer="95"/>
+</segment>
+</net>
+<net name="TX_ON" class="0">
+<segment>
+<pinref part="U3" gate="G$1" pin="TXON"/>
+<wire x1="205.74" y1="111.76" x2="210.82" y2="111.76" width="0.1524" layer="91"/>
+<label x="210.82" y="111.76" size="1.778" layer="95"/>
+</segment>
+</net>
+<net name="5V_BUS" class="0">
+<segment>
+<pinref part="R8" gate="G$1" pin="2"/>
+<wire x1="220.98" y1="121.92" x2="226.06" y2="121.92" width="0.1524" layer="91"/>
+<label x="226.06" y="121.92" size="1.778" layer="95"/>
+</segment>
+</net>
+<net name="SDN" class="0">
+<segment>
+<pinref part="U3" gate="G$1" pin="SDN"/>
+<wire x1="167.64" y1="106.68" x2="162.56" y2="106.68" width="0.1524" layer="91"/>
+<label x="157.48" y="106.68" size="1.778" layer="95"/>
+</segment>
+</net>
+<net name="N$9" class="0">
+<segment>
+<pinref part="R8" gate="G$1" pin="1"/>
+<wire x1="210.82" y1="121.92" x2="205.74" y2="121.92" width="0.1524" layer="91"/>
+<pinref part="U3" gate="G$1" pin="VCC"/>
+</segment>
+</net>
+<net name="N$10" class="0">
+<segment>
+<pinref part="R9" gate="G$1" pin="1"/>
+<pinref part="U4" gate="G$1" pin="3V3"/>
+<wire x1="210.82" y1="63.5" x2="205.74" y2="63.5" width="0.1524" layer="91"/>
+</segment>
+</net>
+<net name="GPS_GND" class="0">
+<segment>
+<pinref part="R6" gate="G$1" pin="1"/>
+<wire x1="58.42" y1="63.5" x2="55.88" y2="63.5" width="0.1524" layer="91"/>
+<label x="55.88" y="63.5" size="1.778" layer="95" rot="MR0"/>
+</segment>
+<segment>
 <pinref part="U6" gate="G$1" pin="GND_RF"/>
 <wire x1="58.42" y1="88.9" x2="58.42" y2="81.28" width="0.1524" layer="91"/>
@@
 <label x="88.9" y="88.9" size="1.778" layer="95" rot="MR270"/>
 </segment>
-<segment>
-<pinref part="R6" gate="G$1" pin="1"/>
-<wire x1="58.42" y1="63.5" x2="55.88" y2="63.5" width="0.1524" layer="91"/>
-<label x="55.88" y="63.5" size="1.778" layer="95" rot="MR0"/>
-</segment>
-</net>
-<net name="UART5_RXD" class="0">
-<segment>
-<pinref part="U6" gate="G$1" pin="GPS_RXDO"/>
-<wire x1="109.22" y1="121.92" x2="121.92" y2="121.92" width="0.1524" layer="91"/>
-<label x="114.3" y="121.92" size="1.778" layer="95"/>
-</segment>
-</net>
-<net name="DIO1" class="0">
-<segment>
-<pinref part="U3" gate="G$1" pin="GPIO_1"/>
-<wire x1="205.74" y1="132.08" x2="210.82" y2="132.08" width="0.1524" layer="91"/>
-<label x="210.82" y="132.08" size="1.778" layer="95"/>
-</segment>
-<segment>
-<pinref part="U4" gate="G$1" pin="DIO1"/>
-<wire x1="205.74" y1="73.66" x2="210.82" y2="73.66" width="0.1524" layer="91"/>
-<label x="210.82" y="73.66" size="1.778" layer="95"/>
-</segment>
-</net>
-<net name="NIRQ" class="0">
-<segment>
-<pinref part="U3" gate="G$1" pin="NIRQ"/>
-<wire x1="167.64" y1="111.76" x2="162.56" y2="111.76" width="0.1524" layer="91"/>
-<label x="157.48" y="111.76" size="1.778" layer="95"/>
-</segment>
-</net>
-<net name="RX_ON" class="0">
-<segment>
-<pinref part="U3" gate="G$1" pin="RXON"/>
-<wire x1="205.74" y1="116.84" x2="210.82" y2="116.84" width="0.1524" layer="91"/>
-<label x="210.82" y="116.84" size="1.778" layer="95"/>
-</segment>
-</net>
-<net name="TX_ON" class="0">
-<segment>
-<pinref part="U3" gate="G$1" pin="TXON"/>
-<wire x1="205.74" y1="111.76" x2="210.82" y2="111.76" width="0.1524" layer="91"/>
-<label x="210.82" y="111.76" size="1.778" layer="95"/>
-</segment>
-</net>
-<net name="5V_BUS" class="0">
-<segment>
-<pinref part="R8" gate="G$1" pin="2"/>
-<wire x1="220.98" y1="121.92" x2="226.06" y2="121.92" width="0.1524" layer="91"/>
-<label x="226.06" y="121.92" size="1.778" layer="95"/>
-</segment>
-</net>
-<net name="SDN" class="0">
-<segment>
-<pinref part="U3" gate="G$1" pin="SDN"/>
-<wire x1="167.64" y1="106.68" x2="162.56" y2="106.68" width="0.1524" layer="91"/>
-<label x="157.48" y="106.68" size="1.778" layer="95"/>
-</segment>
-</net>
-<net name="N$9" class="0">
-<segment>
-<pinref part="R8" gate="G$1" pin="1"/>
-<wire x1="210.82" y1="121.92" x2="205.74" y2="121.92" width="0.1524" layer="91"/>
-<pinref part="U3" gate="G$1" pin="VCC"/>
-</segment>
-</net>
-<net name="N$10" class="0">
-<segment>
-<pinref part="R9" gate="G$1" pin="1"/>
-<pinref part="U4" gate="G$1" pin="3V3"/>
-<wire x1="210.82" y1="63.5" x2="205.74" y2="63.5" width="0.1524" layer="91"/>
-</segment>
-</net>
+</net>
