File: hardware/Eagle Designs/Battery Board/batteryboard-v2.2 (Eagle)/batteryboard-v2.2.sch (EAGLE design)
At the start: 27 parts, among them J1 1042, J10 MOLEX_503763-0291MOLEX_503763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, J15 MOLEX_503763-0291MOLEX_503763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, J2 1042, J3 1042, J4 1042_SMALLPAD, J5 1042, J6 1042, J7 MOLEX_503763-0291MOLEX_503763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, J8 MOLEX_503763-0291MOLEX_503763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

Commit message: Board updates
Parts:
- added J11: TFM-105-01-L-D-RA, TFM-105-01-L-D-RA:TFM-105-01-L-D-RA
Changed lines of the file:
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@@
 <part name="U$1" library="PC104_holes" deviceset="PC104_HOLES" device=""/>
 <part name="J4" library="Keystone_Electronics_1042" deviceset="1042_SMALLPAD" device=""/>
+<part name="J11" library="TFM-105-01-L-D-RA" deviceset="TFM-105-01-L-D-RA" device=""/>
 </parts>
 <sheets>
@@
 <attribute name="VALUE" x="-124.2314" y="99.2886" size="2.0828" layer="96" ratio="6" rot="SR0"/>
 </instance>
+<instance part="J11" gate="G$1" x="-35.56" y="83.82" smashed="yes">
+<attribute name="NAME" x="-43.68" y="91.44" size="1.778" layer="95"/>
+<attribute name="VALUE" x="-43.18" y="73.66" size="1.778" layer="96"/>
+</instance>
 </instances>
