File: hardware/Eagle Designs/Battery Board/batteryboard-v2.2 (KiCad)/_autosave-batteryboard.sch (KiCad schematic (older format))
At the start: 37 parts, among them J1 KEYSTONE-1042, J10 Conn_01x02_Female, J11 5037630291, J12 Screw_Terminal_01x01, J2 KEYSTONE-1042, J3 KEYSTONE-1042, J4 KEYSTONE-1042, J5 KEYSTONE-1042, J6 KEYSTONE-1042, J7 Conn_01x02_Female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

Commit message: Board updates
Connections:
- net labels added: CONN+
- wire segments 86 -> 88
Changed lines of the file:
@@
 	7800 3500 7950 3500
 Wire Wire Line
-	7800 3500 7800 3250
-Wire Wire Line
 	7800 3250 7950 3250
-Connection ~ 7800 3500
 Wire Wire Line
 	6950 3250 7250 3250
-Wire Wire Line
-	7600 3400 7950 3400
 Wire Wire Line
 	7600 3400 7600 3750
 Wire Wire Line
 	7600 3750 7950 3750
-Connection ~ 7600 3400
 Wire Wire Line
 	7600 3750 7600 3950
@@
 Wire Wire Line
 	7600 3150 7600 3250
-Connection ~ 7600 3250
-Wire Wire Line
-	7600 3250 7600 3400
 Text Notes 8250 5850 0    50   ~ 0
 Temp Sensor\n
@@
 Wire Wire Line
 	5150 7300 4850 7300
-Wire Wire Line
-	7600 3150 7900 3150
 $Comp
 L Connector:Conn_01x02_Female J7
@@
 	1    0    0    -1
 $EndComp
-Text Label 7900 3000 0    50   ~ 0
+Wire Wire Line
+	7600 3150 7950 3150
+Text Label 8500 2950 0    50   ~ 0
 CONN
 Wire Wire Line
-	7900 3150 7900 3000
-Connection ~ 7900 3150
+	7950 3150 8500 3150
 Wire Wire Line
-	7900 3150 7950 3150
+	8500 3150 8500 2950
+Connection ~ 7950 3150
+Text Label 9100 3400 0    50   ~ 0
+CONN+
+Wire Wire Line
+	7600 3400 7800 3400
+Wire Wire Line
+	7800 3250 7800 3400
+Connection ~ 7800 3400
+Wire Wire Line
+	7800 3400 7950 3400
+Wire Wire Line
+	9100 3400 7950 3400
+Connection ~ 7950 3400
+Wire Wire Line
+	7950 3400 7800 3400
 $EndSCHEMATC
