File: hardware/Eagle Designs/Battery Board/batteryboard-v2.2 (KiCad)/batteryboard.kicad_pcb (KiCad board)
At the start: 2 copper layers, 95.9 x 90.2 mm, 44 parts, among them J1 KEYSTONE-1042, J10 Conn_01x02_Female, J11 5037630291, J12 Screw_Terminal_01x01, J2 KEYSTONE-1042, J3 KEYSTONE-1042, J4 KEYSTONE-1042, J5 KEYSTONE-1042, J6 KEYSTONE-1042, J7 Conn_01x02_Female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

Commit message: Board updates
Connections:
- J10 pad 2: Net-(J10-Pad2) -> /CONN
- J7 pad 1: Net-(J10-Pad2) -> /CONN
- J7 pad 2: PACK- -> /CONN+
- J8 pad 1: Net-(J10-Pad2) -> /CONN+
- J9 pad 1: Net-(J10-Pad2) -> /CONN+
- J9 pad 3: Net-(J10-Pad2) -> /CONN+
Routing:
- net Net-(J10-Pad2): track 40.4 -> 0.00 mm
- net /CONN+: track 0.00 -> 32.5 mm
- net /CONN: track 0.00 -> 8.55 mm
