File: hardware/Eagle Designs/Battery Board/batteryboard-v3.0/Battery_Board_v3.0.brd (EAGLE design)
At the start: 95.9 x 90.2 mm, 23 parts, among them J1 1042, J2 1042, J3 1042, J4 1042_SMALLPAD, J5 1042, J6 1042, J7 MOLEX_503763-0291MOLEX_503763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, J8 MOLEX_503763-0291MOLEX_503763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, Q1 IRF7458TRPBF, Q2 IRF7458TRPBF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

Commit message: Battery Board V3 Changes
Parts:
- moved U2 0.78 mm to (5.10, 26.3)
Connections:
- removed net GND: H1.17, H1.19, H1.20, H1.21, H1.22, H1.42
- net PACK-: now also H1.17, H1.19, H1.20, H1.21, H1.22, H1.42
Routing:
- net 3V3_BUS: track 138.7 -> 150.5 mm
- net I2C1_SCL: track 75.1 -> 79.6 mm
- net I2C1_SDA: track 70.7 -> 72.4 mm

Commit message: Board updates
Parts:
- removed H1: TFM-130-01-L-D-RA, TFM-130-01-L-D-RA:60_PIN
- U$1: value PC104_HOLES -> V2_BOARD_60PIN; device PC104_holes:PC104_HOLES -> Artemis v2 board:PC104_WCONN_BACKPLANE_HEADER
- moved U$1 130.1 mm to (-92.9, -0.30), turned to 0 degrees
Connections:
- removed net 12V_SW1: H1.18
- removed net 5V_BUS: H1.3, H1.4
- removed net BATT_CHRG: H1.15, H1.16
- removed net BURN1: H1.14
- removed net BURN2: H1.13
- removed net CE0_N: H1.49
- removed net CE1_N: H1.48
- removed net I2C2_SCL: H1.24
- removed net I2C2_SDA: H1.23
- removed net MISO: H1.51
- removed net MOSI: H1.52
- removed net PDU_UART4_RX: H1.59
- removed net PDU_UART4_TX: H1.60
- removed net RX+: H1.38
- removed net RX-: H1.37
- removed net SCLK: H1.50
- removed net SOLAR_IN: H1.34
- removed net SOLAR_IN2: H1.33
- removed net SPI1_D0: H1.45
- removed net SPI1_D1: H1.46
- removed net SPI1_SCLK: H1.47
- removed net SWCLK: H1.43
- removed net SWDIO: H1.41
- removed net SW_3V3_1: H1.12
- removed net SW_3V3_2: H1.11
- removed net SW_5V_1: H1.8
- removed net SW_5V_2: H1.7
- removed net SW_5V_3: H1.10
- removed net SW_5V_4: H1.9
- removed net TRQ_1A: H1.32
- removed net TRQ_1B: H1.31
- removed net TRQ_2A: H1.30
- removed net TRQ_2B: H1.29
- removed net TRQ_3A: H1.28
- removed net TRQ_3B: H1.27
- removed net TRQ_4A: H1.26
- removed net TRQ_4B: H1.25
- removed net TX+: H1.40
- removed net TX+2: H1.36
- removed net TX-: H1.39
- removed net TX-2: H1.35
- removed net T_CS1: H1.44
- removed net UART2_RX: H1.57
- removed net UART2_TX: H1.58
- removed net USB_D+: H1.55
- removed net USB_D-: H1.56
- removed net VBATT: H1.1
- net 3V3_BUS: no longer H1.5, H1.6
- net I2C1_SCL: no longer H1.53
- net I2C1_SDA: no longer H1.54
- net PACK: no longer H1.2
- net PACK-: no longer H1.17, H1.19, H1.20, H1.21, H1.22, H1.42
Routing:
- net I2C1_SDA: track 72.4 -> 42.0 mm
- net PACK: track 11.0 -> 7.41 mm
- net 3V3_BUS: track 150.5 -> 150.0 mm
Other:
- board size 95.9 x 90.2 mm -> 90.2 x 95.5 mm
